Commit message: Work on source code

File: midterm/part_b/source_code/test.urdf (robot description, URDF)
Before this commit: robot pepe, 5 links, 4 joints
Links:
- removed link 12
- removed link 13
- removed link 24
- added link 14, mass 1.4236602665548779; collision cylinder length=1.9371726045358948 radius=0.48366435999041024; visual cylinder length=1.9371726045358948 radius=0.48366435999041024
- added link 17, mass 1.4236602665548779; collision cylinder length=1.9371726045358948 radius=0.48366435999041024; visual cylinder length=1.9371726045358948 radius=0.48366435999041024
- added link 22, mass 0.010644158600718915; collision cylinder length=0.13523224557648672 radius=0.15828530679075792; visual cylinder length=0.13523224557648672 radius=0.15828530679075792
- added link 23, mass 0.010644158600718915; collision cylinder length=0.13523224557648672 radius=0.15828530679075792; visual cylinder length=0.13523224557648672 radius=0.15828530679075792
- added link 25, mass 0.010644158600718915; collision cylinder length=0.13523224557648672 radius=0.15828530679075792; visual cylinder length=0.13523224557648672 radius=0.15828530679075792
- added link 26, mass 0.010644158600718915; collision cylinder length=0.13523224557648672 radius=0.15828530679075792; visual cylinder length=0.13523224557648672 radius=0.15828530679075792
- added link 28, mass 0.010644158600718915; collision cylinder length=0.13523224557648672 radius=0.15828530679075792; visual cylinder length=0.13523224557648672 radius=0.15828530679075792
- added link 29, mass 0.010644158600718915; collision cylinder length=0.13523224557648672 radius=0.15828530679075792; visual cylinder length=0.13523224557648672 radius=0.15828530679075792
- link 0: mass 0.08882193011447076 -> 0.011174829638357359; geometry collision cylinder length=1.3063443781598538 radius=0.052181514386424266; visual cylinder length=1.3063443781598538 radius=0.052181514386424266
- link 11: mass 1.3629571017358157 -> 1.4236602665548779; geometry collision cylinder length=1.9371726045358948 radius=0.48366435999041024; visual cylinder length=1.9371726045358948 radius=0.48366435999041024
Joints:
- removed joint 12_to_0
- removed joint 13_to_0
- removed joint 24_to_0
- added joint 14_to_0: type revolute, parent 0, child 14, origin xyz=0.010830985181975339 0.631308358414573 0.3061320972843057 rpy=13.02364934886986 4.5014198676762085 5.368744709092928, axis 1 0 0, limit lower=3.1415 upper=-3.1415 effort=1 velocity=1
- added joint 17_to_0: type revolute, parent 0, child 17, origin xyz=0.010830985181975339 0.631308358414573 0.3061320972843057 rpy=17.364865798493145 4.5014198676762085 5.368744709092928, axis 1 0 0, limit lower=3.1415 upper=-3.1415 effort=1 velocity=1
- added joint 22_to_11: type revolute, parent 11, child 22, origin xyz=0.9685756510168184 0.5696210528788638 0.37088863911264824 rpy=2.6278403408763404 0.8117556711956565 3.330975315413971, axis 0 1 0, limit lower=3.1415 upper=-3.1415 effort=1 velocity=1
- added joint 23_to_11: type revolute, parent 11, child 23, origin xyz=0.9685756510168184 0.5696210528788638 0.37088863911264824 rpy=3.9417605113145107 0.8117556711956565 3.330975315413971, axis 0 1 0, limit lower=3.1415 upper=-3.1415 effort=1 velocity=1
- added joint 25_to_14: type revolute, parent 14, child 25, origin xyz=0.9685756510168184 0.5696210528788638 0.37088863911264824 rpy=2.6278403408763404 0.8117556711956565 3.330975315413971, axis 0 1 0, limit lower=3.1415 upper=-3.1415 effort=1 velocity=1
- added joint 26_to_14: type revolute, parent 14, child 26, origin xyz=0.9685756510168184 0.5696210528788638 0.37088863911264824 rpy=3.9417605113145107 0.8117556711956565 3.330975315413971, axis 0 1 0, limit lower=3.1415 upper=-3.1415 effort=1 velocity=1
- added joint 28_to_17: type revolute, parent 17, child 28, origin xyz=0.9685756510168184 0.5696210528788638 0.37088863911264824 rpy=2.6278403408763404 0.8117556711956565 3.330975315413971, axis 0 1 0, limit lower=3.1415 upper=-3.1415 effort=1 velocity=1
- added joint 29_to_17: type revolute, parent 17, child 29, origin xyz=0.9685756510168184 0.5696210528788638 0.37088863911264824 rpy=3.9417605113145107 0.8117556711956565 3.330975315413971, axis 0 1 0, limit lower=3.1415 upper=-3.1415 effort=1 velocity=1
- joint 11_to_0: axis 0 0 1 -> 1 0 0; origin xyz=0.13758607675745194 0.9350807390271525 0.7734982986138889 rpy=1.1448832225386056 4.335027266637536 1.6623373384868418 -> xyz=0.010830985181975339 0.631308358414573 0.3061320972843057 rpy=8.682432899246573 4.5014198676762085 5.368744709092928

Commit message: Touch up code base

File: midterm/part_b/source_code/test.urdf (robot description, URDF)
Before this commit: robot pepe, 10 links, 9 joints
Links:
- removed link 14
- removed link 17
- removed link 22
- removed link 25
- removed link 26
- removed link 28
- removed link 29
- added link 12, mass 1.9545196365709276; collision cylinder length=0.835509285331441 radius=0.8629178292703552; visual cylinder length=0.835509285331441 radius=0.8629178292703552
- added link 24, mass 0.5772457567525413; collision cylinder length=1.077876471559702 radius=0.4128772393555715; visual cylinder length=1.077876471559702 radius=0.4128772393555715
- link 0: mass 0.011174829638357359 -> 0.0098846122531829; geometry collision cylinder length=1.6112201748019956 radius=0.044190349553533625; visual cylinder length=1.6112201748019956 radius=0.044190349553533625
- link 11: mass 1.4236602665548779 -> 1.9545196365709276; geometry collision cylinder length=0.835509285331441 radius=0.8629178292703552; visual cylinder length=0.835509285331441 radius=0.8629178292703552
- link 23: mass 0.010644158600718915 -> 0.5772457567525413; geometry collision cylinder length=1.077876471559702 radius=0.4128772393555715; visual cylinder length=1.077876471559702 radius=0.4128772393555715
Joints:
- removed joint 14_to_0
- removed joint 17_to_0
- removed joint 22_to_11
- removed joint 23_to_11
- removed joint 25_to_14
- removed joint 26_to_14
- removed joint 28_to_17
- removed joint 29_to_17
- added joint 12_to_0: type revolute, parent 0, child 12, origin xyz=0.15806658421273412 0.8702749981053901 0.09008178169454528 rpy=11.022399058515726 1.286696162537153 2.047689694017483, axis 0 1 0, limit lower=3.1415 upper=-3.1415 effort=1 velocity=1
- added joint 23_to_0: type revolute, parent 0, child 23, origin xyz=0.5962960219636788 0.4144361426774621 0.41810579585382257 rpy=6.68549386934984 2.7954775727547405 2.225478645018462, axis 0 1 0, limit lower=3.1415 upper=-3.1415 effort=1 velocity=1
- added joint 24_to_0: type revolute, parent 0, child 24, origin xyz=0.5962960219636788 0.4144361426774621 0.41810579585382257 rpy=8.3568673366873 2.7954775727547405 2.225478645018462, axis 0 1 0, limit lower=3.1415 upper=-3.1415 effort=1 velocity=1
- joint 11_to_0: axis 1 0 0 -> 0 1 0; origin xyz=0.010830985181975339 0.631308358414573 0.3061320972843057 rpy=8.682432899246573 4.5014198676762085 5.368744709092928 -> xyz=0.15806658421273412 0.8702749981053901 0.09008178169454528 rpy=7.3482660390104835 1.286696162537153 2.047689694017483

Commit message: Work on project

File: midterm/part_b/source_code/test.urdf (robot description, URDF)
Before this commit: robot pepe, 5 links, 4 joints
Links:
- removed link 24
- link 0: mass 0.0098846122531829 -> 0.11135622718705726; geometry collision cylinder length=0.1160686038304839 radius=0.5526178865973497; visual cylinder length=0.1160686038304839 radius=0.5526178865973497
- link 11: mass 1.9545196365709276 -> 0.04014940331203455; geometry collision cylinder length=0.7169652542622151 radius=0.13351054128965612; visual cylinder length=0.7169652542622151 radius=0.13351054128965612
- link 12: mass 1.9545196365709276 -> 0.04014940331203455; geometry collision cylinder length=0.7169652542622151 radius=0.13351054128965612; visual cylinder length=0.7169652542622151 radius=0.13351054128965612
- link 23: mass 0.5772457567525413 -> 0.13649649628798102; geometry collision cylinder length=1.7414681952463393 radius=0.1579530592767211; visual cylinder length=1.7414681952463393 radius=0.1579530592767211
Joints:
- removed joint 24_to_0
- joint 11_to_0: axis 0 1 0 -> 1 0 0; origin xyz=0.15806658421273412 0.8702749981053901 0.09008178169454528 rpy=7.3482660390104835 1.286696162537153 2.047689694017483 -> xyz=0.44426846050209123 0.24223650318443568 0.8636264996805906 rpy=1.390943851488836 4.743816113870655 2.778066593216199
- joint 12_to_0: axis 0 1 0 -> 1 0 0; origin xyz=0.15806658421273412 0.8702749981053901 0.09008178169454528 rpy=11.022399058515726 1.286696162537153 2.047689694017483 -> xyz=0.44426846050209123 0.24223650318443568 0.8636264996805906 rpy=2.086415777233254 4.743816113870655 2.778066593216199
- joint 23_to_0: origin xyz=0.5962960219636788 0.4144361426774621 0.41810579585382257 rpy=6.68549386934984 2.7954775727547405 2.225478645018462 -> xyz=0.7070234678620229 0.9377480516019508 0.5796473697877225 rpy=14.044334340705712 1.8036339998062194 5.601262011292839

Commit message: WOrk on project

File: midterm/part_b/source_code/test.urdf (robot description, URDF)
Before this commit: robot pepe, 121 links, 120 joints
Links:
- removed link 10104
- removed link 10105
- removed link 10106
- removed link 10113
- removed link 10114
- removed link 10115
- removed link 11120
- removed link 120
- removed link 1270
- removed link 1279
- removed link 1288
- removed link 1371
- removed link 1375
- removed link 1380
- removed link 1384
- removed link 1389
- removed link 139
- removed link 1393
- removed link 1461
- removed link 1462
- removed link 1464
- removed link 1465
- removed link 1467
- removed link 1468
- removed link 1572
- removed link 1573
- removed link 1574
- removed link 1576
- removed link 1577
- removed link 1578
- removed link 1581
- removed link 1582
- removed link 1583
- removed link 1585
- removed link 1586
- removed link 1587
- removed link 1590
- removed link 1591
- removed link 1592
- removed link 1594
- removed link 1595
- removed link 1596
- removed link 16107
- removed link 16108
- removed link 16116
- removed link 16117
- removed link 1797
- removed link 1798
- removed link 1799
- removed link 18118
- removed link 18119
- removed link 1912
- removed link 1913
- removed link 1918
- removed link 1919
- removed link 1925
- removed link 1926
- removed link 1931
- removed link 1932
- removed link 1937
- removed link 1938
- removed link 1944
- removed link 1945
- removed link 1950
- removed link 1951
- removed link 1956
- removed link 1957
- removed link 196
- removed link 197
- removed link 258
- removed link 359
- removed link 414
- removed link 42
- removed link 421
- removed link 427
- removed link 433
- removed link 440
- removed link 446
- removed link 452
- removed link 48
- removed link 560
- removed link 563
- removed link 566
- removed link 669
- removed link 710
- removed link 711
- removed link 715
- removed link 716
- removed link 717
- removed link 722
- removed link 723
- removed link 724
- removed link 728
- removed link 729
- removed link 73
- removed link 730
- removed link 734
- removed link 735
- removed link 736
- removed link 74
- removed link 741
- removed link 742
- removed link 743
- removed link 747
- removed link 748
- removed link 749
- removed link 75
- removed link 753
- removed link 754
- removed link 755
- removed link 79
- removed link 8100
- removed link 8109
- removed link 9101
- removed link 9102
- removed link 9103
- removed link 9110
- removed link 9111
- removed link 9112
- added link 22, mass 1.0591589788813363; collision cylinder length=1.4356933729939825 radius=0.484590383967605; visual cylinder length=1.4356933729939825 radius=0.484590383967605
- added link 23, mass 1.0591589788813363; collision cylinder length=1.4356933729939825 radius=0.484590383967605; visual cylinder length=1.4356933729939825 radius=0.484590383967605
- link 0: mass 0.4803369081357246 -> 0.0012980589069353638; geometry collision cylinder length=0.942222838912345 radius=0.020940905207326943; visual cylinder length=0.942222838912345 radius=0.020940905207326943
- link 11: mass 0.5868061104449045 -> 1.9953709268606092; geometry collision cylinder length=1.9974540602296298 radius=0.5638953117657445; visual cylinder length=1.9974540602296298 radius=0.5638953117657445
Joints:
- removed joint 10104_to_8100
- removed joint 10105_to_8100
- removed joint 10106_to_8100
- removed joint 10113_to_8109
- removed joint 10114_to_8109
- removed joint 10115_to_8109
- removed joint 11120_to_0
- removed joint 120_to_0
- removed joint 1270_to_669
- removed joint 1279_to_669
- removed joint 1288_to_669
- removed joint 1371_to_1270
- removed joint 1375_to_1270
- removed joint 1380_to_1279
- removed joint 1384_to_1279
- removed joint 1389_to_1288
- removed joint 1393_to_1288
- removed joint 139_to_0
- removed joint 1461_to_560
- removed joint 1462_to_560
- removed joint 1464_to_563
- removed joint 1465_to_563
- removed joint 1467_to_566
- removed joint 1468_to_566
- removed joint 1572_to_1371
- removed joint 1573_to_1371
- removed joint 1574_to_1371
- removed joint 1576_to_1375
- removed joint 1577_to_1375
- removed joint 1578_to_1375
- removed joint 1581_to_1380
- removed joint 1582_to_1380
- removed joint 1583_to_1380
- removed joint 1585_to_1384
- removed joint 1586_to_1384
- removed joint 1587_to_1384
- removed joint 1590_to_1389
- removed joint 1591_to_1389
- removed joint 1592_to_1389
- removed joint 1594_to_1393
- removed joint 1595_to_1393
- removed joint 1596_to_1393
- removed joint 16107_to_8100
- removed joint 16108_to_8100
- removed joint 16116_to_8109
- removed joint 16117_to_8109
- removed joint 1797_to_669
- removed joint 1798_to_669
- removed joint 1799_to_669
- removed joint 18118_to_258
- removed joint 18119_to_258
- removed joint 1912_to_48
- removed joint 1913_to_48
- removed joint 1918_to_414
- removed joint 1919_to_414
- removed joint 1925_to_421
- removed joint 1926_to_421
- removed joint 1931_to_427
- removed joint 1932_to_427
- removed joint 1937_to_433
- removed joint 1938_to_433
- removed joint 1944_to_440
- removed joint 1945_to_440
- removed joint 1950_to_446
- removed joint 1951_to_446
- removed joint 1956_to_452
- removed joint 1957_to_452
- removed joint 196_to_42
- removed joint 197_to_42
- removed joint 258_to_0
- removed joint 359_to_258
- removed joint 414_to_11
- removed joint 421_to_120
- removed joint 427_to_120
- removed joint 42_to_11
- removed joint 433_to_120
- removed joint 440_to_139
- removed joint 446_to_139
- removed joint 452_to_139
- removed joint 48_to_11
- removed joint 560_to_359
- removed joint 563_to_359
- removed joint 566_to_359
- removed joint 669_to_258
- removed joint 710_to_48
- removed joint 711_to_48
- removed joint 715_to_414
- removed joint 716_to_414
- removed joint 717_to_414
- removed joint 722_to_421
- removed joint 723_to_421
- removed joint 724_to_421
- removed joint 728_to_427
- removed joint 729_to_427
- removed joint 730_to_427
- removed joint 734_to_433
- removed joint 735_to_433
- removed joint 736_to_433
- removed joint 73_to_42
- removed joint 741_to_440
- removed joint 742_to_440
- removed joint 743_to_440
- removed joint 747_to_446
- removed joint 748_to_446
- removed joint 749_to_446
- removed joint 74_to_42
- removed joint 753_to_452
- removed joint 754_to_452
- removed joint 755_to_452
- removed joint 75_to_42
- removed joint 79_to_48
- removed joint 8100_to_258
- removed joint 8109_to_258
- removed joint 9101_to_8100
- removed joint 9102_to_8100
- removed joint 9103_to_8100
- removed joint 9110_to_8109
- removed joint 9111_to_8109
- removed joint 9112_to_8109
- added joint 22_to_11: type revolute, parent 11, child 22, origin xyz=0.30185808897508215 0.3525499804151325 0.7831233119247555 rpy=3.804460657035247 1.7345844943793804 3.946440847852103, axis 0 1 0, limit lower=3.1415 upper=-3.1415 effort=1 velocity=1
- added joint 23_to_11: type revolute, parent 11, child 23, origin xyz=0.30185808897508215 0.3525499804151325 0.7831233119247555 rpy=5.7066909855528705 1.7345844943793804 3.946440847852103, axis 0 1 0, limit lower=3.1415 upper=-3.1415 effort=1 velocity=1
- joint 11_to_0: axis 1 0 0 -> 0 0 1; origin xyz=0.30409346612201027 0.4020096373369314 0.503608975842264 rpy=0.08248414446588753 2.8119372169068653 1.1269094142387204 -> xyz=0.1111167058687742 0.21960449127547765 0.7162651618899991 rpy=10.948734228388998 1.8753530056298873 4.716899293222515
