Commit message: Finish code walkthrough

File: midterm/part_b/source_code/temp0.urdf (robot description, URDF)
Before this commit: robot pepe, 4 links, 3 joints
Links:
- link 0: mass 3.1454160229753874 -> 0.5636468459567316; geometry collision cylinder length=0.8755907652356707 radius=0.45266614839352026; visual cylinder length=0.8755907652356707 radius=0.45266614839352026
- link 11: mass 2.856802280917818 -> 1.5813387482445305; geometry collision cylinder length=1.0926837629257198 radius=0.6787194192735374; visual cylinder length=1.0926837629257198 radius=0.6787194192735374
- link 12: mass 2.856802280917818 -> 1.5813387482445305; geometry collision cylinder length=1.0926837629257198 radius=0.6787194192735374; visual cylinder length=1.0926837629257198 radius=0.6787194192735374
- link 13: mass 2.856802280917818 -> 1.5813387482445305; geometry collision cylinder length=1.0926837629257198 radius=0.6787194192735374; visual cylinder length=1.0926837629257198 radius=0.6787194192735374
Joints:
- joint 11_to_0: axis 1 0 0 -> 0 0 1; origin xyz=0.1462641576616387 0.5572290704684391 0.8285118940376992 rpy=9.822124079454426 4.041582349174072 4.382430559563875 -> xyz=0.8307121265962392 0.9735949054547904 0.24192579126684943 rpy=7.171165116166609 0.06333445163193102 4.001400464474772
- joint 12_to_0: axis 1 0 0 -> 0 0 1; origin xyz=0.1462641576616387 0.5572290704684391 0.8285118940376992 rpy=14.733186119181639 4.041582349174072 4.382430559563875 -> xyz=0.8307121265962392 0.9735949054547904 0.24192579126684943 rpy=10.756747674249914 0.06333445163193102 4.001400464474772
- joint 13_to_0: axis 1 0 0 -> 0 0 1; origin xyz=0.1462641576616387 0.5572290704684391 0.8285118940376992 rpy=19.64424815890885 4.041582349174072 4.382430559563875 -> xyz=0.8307121265962392 0.9735949054547904 0.24192579126684943 rpy=14.342330232333218 0.06333445163193102 4.001400464474772

File: midterm/part_b/source_code/test.urdf (robot description, URDF)
Before this commit: robot pepe, 4 links, 3 joints
Links:
- removed link 23
- added link 13, mass 1.1506211025735562; collision cylinder length=0.5625772901796258 radius=0.8068636167950674; visual cylinder length=0.5625772901796258 radius=0.8068636167950674
- added link 15, mass 1.1506211025735562; collision cylinder length=0.5625772901796258 radius=0.8068636167950674; visual cylinder length=0.5625772901796258 radius=0.8068636167950674
- added link 24, mass 0.1743645496166827; collision cylinder length=0.15441705586968713 radius=0.599523934459773; visual cylinder length=0.15441705586968713 radius=0.599523934459773
- added link 26, mass 0.1743645496166827; collision cylinder length=0.15441705586968713 radius=0.599523934459773; visual cylinder length=0.15441705586968713 radius=0.599523934459773
- link 0: mass 0.0012980589069353638 -> 0.0006491701219059603; geometry collision cylinder length=1.1226638615419493 radius=0.013566863446804911; visual cylinder length=1.1226638615419493 radius=0.013566863446804911
- link 11: mass 1.9953709268606092 -> 1.1506211025735562; geometry collision cylinder length=0.5625772901796258 radius=0.8068636167950674; visual cylinder length=0.5625772901796258 radius=0.8068636167950674
- link 22: mass 1.0591589788813363 -> 0.1743645496166827; geometry collision cylinder length=0.15441705586968713 radius=0.599523934459773; visual cylinder length=0.15441705586968713 radius=0.599523934459773
Joints:
- removed joint 23_to_11
- added joint 13_to_0: type revolute, parent 0, child 13, origin xyz=0.18977128553073197 0.5336053814382133 0.17036618091553735 rpy=7.08169284061338 1.9845007485072967 1.53768567894434, axis 0 0 1, limit lower=3.1415 upper=-3.1415 effort=1 velocity=1
- added joint 15_to_0: type revolute, parent 0, child 15, origin xyz=0.18977128553073197 0.5336053814382133 0.17036618091553735 rpy=9.44225712081784 1.9845007485072967 1.53768567894434, axis 0 0 1, limit lower=3.1415 upper=-3.1415 effort=1 velocity=1
- added joint 24_to_13: type revolute, parent 13, child 24, origin xyz=0.6287796269892859 0.4798738006784883 0.6636635622644665 rpy=9.519351475367962 1.7503012391596664 1.6078731196274874, axis 0 0 1, limit lower=3.1415 upper=-3.1415 effort=1 velocity=1
- added joint 26_to_15: type revolute, parent 15, child 26, origin xyz=0.6287796269892859 0.4798738006784883 0.6636635622644665 rpy=9.519351475367962 1.7503012391596664 1.6078731196274874, axis 0 0 1, limit lower=3.1415 upper=-3.1415 effort=1 velocity=1
- joint 11_to_0: origin xyz=0.1111167058687742 0.21960449127547765 0.7162651618899991 rpy=10.948734228388998 1.8753530056298873 4.716899293222515 -> xyz=0.18977128553073197 0.5336053814382133 0.17036618091553735 rpy=4.72112856040892 1.9845007485072967 1.53768567894434
- joint 22_to_11: axis 0 1 0 -> 0 0 1; origin xyz=0.30185808897508215 0.3525499804151325 0.7831233119247555 rpy=3.804460657035247 1.7345844943793804 3.946440847852103 -> xyz=0.6287796269892859 0.4798738006784883 0.6636635622644665 rpy=9.519351475367962 1.7503012391596664 1.6078731196274874
