Commit message: Work on project

File: midterm/part_b/source_code/my_code/temp0.urdf (robot description, URDF)
Before this commit: robot pepe, 5 links, 4 joints
Links:
- removed link 12
- added link 15, mass 0.594323282278726; collision cylinder length=1.1872376092644017 radius=0.3991789327641704; visual cylinder length=1.1872376092644017 radius=0.3991789327641704
- added link 19, mass 0.594323282278726; collision cylinder length=1.1872376092644017 radius=0.3991789327641704; visual cylinder length=1.1872376092644017 radius=0.3991789327641704
- added link 210, mass 1.1224534124002217; collision cylinder length=0.669974225979638 radius=0.7302644817118741; visual cylinder length=0.669974225979638 radius=0.7302644817118741
- added link 211, mass 1.1224534124002217; collision cylinder length=0.669974225979638 radius=0.7302644817118741; visual cylinder length=0.669974225979638 radius=0.7302644817118741
- added link 212, mass 1.1224534124002217; collision cylinder length=0.669974225979638 radius=0.7302644817118741; visual cylinder length=0.669974225979638 radius=0.7302644817118741
- added link 22, mass 1.1224534124002217; collision cylinder length=0.669974225979638 radius=0.7302644817118741; visual cylinder length=0.669974225979638 radius=0.7302644817118741
- added link 26, mass 1.1224534124002217; collision cylinder length=0.669974225979638 radius=0.7302644817118741; visual cylinder length=0.669974225979638 radius=0.7302644817118741
- added link 27, mass 1.1224534124002217; collision cylinder length=0.669974225979638 radius=0.7302644817118741; visual cylinder length=0.669974225979638 radius=0.7302644817118741
- added link 28, mass 1.1224534124002217; collision cylinder length=0.669974225979638 radius=0.7302644817118741; visual cylinder length=0.669974225979638 radius=0.7302644817118741
- link 0: mass 0.008343661714698665 -> 0.3442880002547839; geometry collision cylinder length=0.10959542754246421 radius=0.9999764888571718; visual cylinder length=0.10959542754246421 radius=0.9999764888571718
- link 11: mass 1.1805110215364507 -> 0.594323282278726; geometry collision cylinder length=1.1872376092644017 radius=0.3991789327641704; visual cylinder length=1.1872376092644017 radius=0.3991789327641704
- link 23: mass 5.217796429387148 -> 1.1224534124002217; geometry collision cylinder length=0.669974225979638 radius=0.7302644817118741; visual cylinder length=0.669974225979638 radius=0.7302644817118741
- link 24: mass 5.217796429387148 -> 1.1224534124002217; geometry collision cylinder length=0.669974225979638 radius=0.7302644817118741; visual cylinder length=0.669974225979638 radius=0.7302644817118741
Joints:
- removed joint 12_to_0
- removed joint 23_to_0
- removed joint 24_to_0
- added joint 15_to_0: type revolute, parent 0, child 15, origin xyz=0.39375438723311196 0.7626037178264388 0.25863347841572515 rpy=8.66839731745303 4.588609673539818 0.1419210292937197, axis 0 1 0, limit lower=3.1415 upper=-3.1415 effort=1 velocity=1
- added joint 19_to_0: type revolute, parent 0, child 19, origin xyz=0.39375438723311196 0.7626037178264388 0.25863347841572515 rpy=11.557863089937372 4.588609673539818 0.1419210292937197, axis 0 1 0, limit lower=3.1415 upper=-3.1415 effort=1 velocity=1
- added joint 210_to_19: type revolute, parent 19, child 210, origin xyz=0.8802687168556907 0.4251184254746059 0.09822746496964774 rpy=0.5613268204832329 4.050807946371586 0.5191958401016188, axis 1 0 0, limit lower=3.1415 upper=-3.1415 effort=1 velocity=1
- added joint 211_to_19: type revolute, parent 19, child 211, origin xyz=0.8802687168556907 0.4251184254746059 0.09822746496964774 rpy=0.8419902307248494 4.050807946371586 0.5191958401016188, axis 1 0 0, limit lower=3.1415 upper=-3.1415 effort=1 velocity=1
- added joint 212_to_19: type revolute, parent 19, child 212, origin xyz=0.8802687168556907 0.4251184254746059 0.09822746496964774 rpy=1.1226536409664658 4.050807946371586 0.5191958401016188, axis 1 0 0, limit lower=3.1415 upper=-3.1415 effort=1 velocity=1
- added joint 22_to_11: type revolute, parent 11, child 22, origin xyz=0.8802687168556907 0.4251184254746059 0.09822746496964774 rpy=0.5613268204832329 4.050807946371586 0.5191958401016188, axis 1 0 0, limit lower=3.1415 upper=-3.1415 effort=1 velocity=1
- added joint 23_to_11: type revolute, parent 11, child 23, origin xyz=0.8802687168556907 0.4251184254746059 0.09822746496964774 rpy=0.8419902307248494 4.050807946371586 0.5191958401016188, axis 1 0 0, limit lower=3.1415 upper=-3.1415 effort=1 velocity=1
- added joint 24_to_11: type revolute, parent 11, child 24, origin xyz=0.8802687168556907 0.4251184254746059 0.09822746496964774 rpy=1.1226536409664658 4.050807946371586 0.5191958401016188, axis 1 0 0, limit lower=3.1415 upper=-3.1415 effort=1 velocity=1
- added joint 26_to_15: type revolute, parent 15, child 26, origin xyz=0.8802687168556907 0.4251184254746059 0.09822746496964774 rpy=0.5613268204832329 4.050807946371586 0.5191958401016188, axis 1 0 0, limit lower=3.1415 upper=-3.1415 effort=1 velocity=1
- added joint 27_to_15: type revolute, parent 15, child 27, origin xyz=0.8802687168556907 0.4251184254746059 0.09822746496964774 rpy=0.8419902307248494 4.050807946371586 0.5191958401016188, axis 1 0 0, limit lower=3.1415 upper=-3.1415 effort=1 velocity=1
- added joint 28_to_15: type revolute, parent 15, child 28, origin xyz=0.8802687168556907 0.4251184254746059 0.09822746496964774 rpy=1.1226536409664658 4.050807946371586 0.5191958401016188, axis 1 0 0, limit lower=3.1415 upper=-3.1415 effort=1 velocity=1
- joint 11_to_0: origin xyz=0.0810917475125349 0.15760646038614268 0.1950018362705248 rpy=6.917068562644353 5.196394829557684 4.873947370565327 -> xyz=0.39375438723311196 0.7626037178264388 0.25863347841572515 rpy=5.778931544968686 4.588609673539818 0.1419210292937197

Commit message: Work on project

File: midterm/part_b/source_code/my_code/temp0.urdf (robot description, URDF)
Before this commit: robot pepe, 13 links, 12 joints
Links:
- removed link 15
- removed link 19
- removed link 210
- removed link 211
- removed link 212
- removed link 24
- removed link 27
- added link 14, mass 0.03102951580780004; collision cylinder length=0.4011584174642282 radius=0.1569114401262658; visual cylinder length=0.4011584174642282 radius=0.1569114401262658
- added link 17, mass 0.03102951580780004; collision cylinder length=0.4011584174642282 radius=0.1569114401262658; visual cylinder length=0.4011584174642282 radius=0.1569114401262658
- added link 25, mass 0.45448627054891244; collision cylinder length=0.3364881694612829 radius=0.655693001120422; visual cylinder length=0.3364881694612829 radius=0.655693001120422
- added link 29, mass 0.45448627054891244; collision cylinder length=0.3364881694612829 radius=0.655693001120422; visual cylinder length=0.3364881694612829 radius=0.655693001120422
- link 0: mass 0.3442880002547839 -> 0.14697746133917491; geometry collision cylinder length=1.6348850655714735 radius=0.1691635619662465; visual cylinder length=1.6348850655714735 radius=0.1691635619662465
- link 11: mass 0.594323282278726 -> 0.03102951580780004; geometry collision cylinder length=0.4011584174642282 radius=0.1569114401262658; visual cylinder length=0.4011584174642282 radius=0.1569114401262658
- link 22: mass 1.1224534124002217 -> 0.45448627054891244; geometry collision cylinder length=0.3364881694612829 radius=0.655693001120422; visual cylinder length=0.3364881694612829 radius=0.655693001120422
- link 23: mass 1.1224534124002217 -> 0.45448627054891244; geometry collision cylinder length=0.3364881694612829 radius=0.655693001120422; visual cylinder length=0.3364881694612829 radius=0.655693001120422
- link 26: mass 1.1224534124002217 -> 0.45448627054891244; geometry collision cylinder length=0.3364881694612829 radius=0.655693001120422; visual cylinder length=0.3364881694612829 radius=0.655693001120422
- link 28: mass 1.1224534124002217 -> 0.45448627054891244; geometry collision cylinder length=0.3364881694612829 radius=0.655693001120422; visual cylinder length=0.3364881694612829 radius=0.655693001120422
Joints:
- removed joint 15_to_0
- removed joint 19_to_0
- removed joint 210_to_19
- removed joint 211_to_19
- removed joint 212_to_19
- removed joint 24_to_11
- removed joint 26_to_15
- removed joint 27_to_15
- removed joint 28_to_15
- added joint 14_to_0: type revolute, parent 0, child 14, origin xyz=0.12660416186520818 0.648604377167844 0.08344684678212422 rpy=4.388183362209325 2.769774899783073 0.8038000893717582, axis 0 1 0, limit lower=3.1415 upper=-3.1415 effort=1 velocity=1
- added joint 17_to_0: type revolute, parent 0, child 17, origin xyz=0.12660416186520818 0.648604377167844 0.08344684678212422 rpy=5.850911149612434 2.769774899783073 0.8038000893717582, axis 0 1 0, limit lower=3.1415 upper=-3.1415 effort=1 velocity=1
- added joint 25_to_14: type revolute, parent 14, child 25, origin xyz=0.03785465984148573 0.7040028254855917 0.23597524873219455 rpy=8.42822902027469 3.7073254045142585 1.4564512245329693, axis 1 0 0, limit lower=3.1415 upper=-3.1415 effort=1 velocity=1
- added joint 26_to_14: type revolute, parent 14, child 26, origin xyz=0.03785465984148573 0.7040028254855917 0.23597524873219455 rpy=12.642343530412035 3.7073254045142585 1.4564512245329693, axis 1 0 0, limit lower=3.1415 upper=-3.1415 effort=1 velocity=1
- added joint 28_to_17: type revolute, parent 17, child 28, origin xyz=0.03785465984148573 0.7040028254855917 0.23597524873219455 rpy=8.42822902027469 3.7073254045142585 1.4564512245329693, axis 1 0 0, limit lower=3.1415 upper=-3.1415 effort=1 velocity=1
- added joint 29_to_17: type revolute, parent 17, child 29, origin xyz=0.03785465984148573 0.7040028254855917 0.23597524873219455 rpy=12.642343530412035 3.7073254045142585 1.4564512245329693, axis 1 0 0, limit lower=3.1415 upper=-3.1415 effort=1 velocity=1
- joint 11_to_0: origin xyz=0.39375438723311196 0.7626037178264388 0.25863347841572515 rpy=5.778931544968686 4.588609673539818 0.1419210292937197 -> xyz=0.12660416186520818 0.648604377167844 0.08344684678212422 rpy=2.925455574806217 2.769774899783073 0.8038000893717582
- joint 22_to_11: origin xyz=0.8802687168556907 0.4251184254746059 0.09822746496964774 rpy=0.5613268204832329 4.050807946371586 0.5191958401016188 -> xyz=0.03785465984148573 0.7040028254855917 0.23597524873219455 rpy=8.42822902027469 3.7073254045142585 1.4564512245329693
- joint 23_to_11: origin xyz=0.8802687168556907 0.4251184254746059 0.09822746496964774 rpy=0.8419902307248494 4.050807946371586 0.5191958401016188 -> xyz=0.03785465984148573 0.7040028254855917 0.23597524873219455 rpy=12.642343530412035 3.7073254045142585 1.4564512245329693

File: midterm/part_b/source_code/my_code/test.urdf (robot description, URDF)
Before this commit: robot pepe, 2 links, 1 joints
Links:
- added link 12, mass 0.11181161068801812; collision cylinder length=0.05584718243022202 radius=0.7983032215789911; visual cylinder length=0.05584718243022202 radius=0.7983032215789911
- added link 13, mass 0.11181161068801812; collision cylinder length=0.05584718243022202 radius=0.7983032215789911; visual cylinder length=0.05584718243022202 radius=0.7983032215789911
- added link 24, mass 0.0005475799489116338; collision cylinder length=0.4542608681033413 radius=0.01958827393542406; visual cylinder length=0.4542608681033413 radius=0.01958827393542406
- added link 25, mass 0.0005475799489116338; collision cylinder length=0.4542608681033413 radius=0.01958827393542406; visual cylinder length=0.4542608681033413 radius=0.01958827393542406
- link 0: mass 0.06967240031004912 -> 1.3201253554439543; geometry collision cylinder length=1.1286729623436214 radius=0.6101668221556736; visual cylinder length=1.1286729623436214 radius=0.6101668221556736
- link 11: mass 1.2317090111199895 -> 0.11181161068801812; geometry collision cylinder length=0.05584718243022202 radius=0.7983032215789911; visual cylinder length=0.05584718243022202 radius=0.7983032215789911
Joints:
- added joint 12_to_0: type revolute, parent 0, child 12, origin xyz=0.41559261142294956 0.1438599694240963 0.29914652633218375 rpy=8.306086401332502 2.4991748170154304 3.895525149863389, axis 0 1 0, limit lower=3.1415 upper=-3.1415 effort=1 velocity=1
- added joint 13_to_0: type revolute, parent 0, child 13, origin xyz=0.41559261142294956 0.1438599694240963 0.29914652633218375 rpy=11.074781868443337 2.4991748170154304 3.895525149863389, axis 0 1 0, limit lower=3.1415 upper=-3.1415 effort=1 velocity=1
- added joint 24_to_0: type revolute, parent 0, child 24, origin xyz=0.6777177586294892 0.3279591849716206 0.5477570993432589 rpy=19.448962758567937 6.255186676264547 6.076207742751965, axis 1 0 0, limit lower=3.1415 upper=-3.1415 effort=1 velocity=1
- added joint 25_to_0: type revolute, parent 0, child 25, origin xyz=0.6777177586294892 0.3279591849716206 0.5477570993432589 rpy=23.338755310281527 6.255186676264547 6.076207742751965, axis 1 0 0, limit lower=3.1415 upper=-3.1415 effort=1 velocity=1
- joint 11_to_0: axis 1 0 0 -> 0 1 0; origin xyz=0.3383974611831103 0.19036004753434088 0.3514409665893894 rpy=3.443162318762247 6.282556988648868 0.6362391480720618 -> xyz=0.41559261142294956 0.1438599694240963 0.29914652633218375 rpy=5.537390934221668 2.4991748170154304 3.895525149863389

Commit message: Work on project

File: midterm/part_b/source_code/my_code/temp0.urdf (robot description, URDF)
Before this commit: robot pepe, 10 links, 9 joints
Links:
- removed link 11
- removed link 14
- removed link 17
- removed link 22
- removed link 23
- removed link 25
- removed link 26
- removed link 28
- removed link 29
- link 0: mass 0.14697746133917491 -> 3.642215640841591; geometry collision cylinder length=1.661534735313683 radius=0.8353205749494185; visual cylinder length=1.661534735313683 radius=0.8353205749494185
Joints:
- removed joint 11_to_0
- removed joint 14_to_0
- removed joint 17_to_0
- removed joint 22_to_11
- removed joint 23_to_11
- removed joint 25_to_14
- removed joint 26_to_14
- removed joint 28_to_17
- removed joint 29_to_17

Commit message: Work on project

File: midterm/part_b/source_code/my_code/temp0.urdf (robot description, URDF)
Before this commit: robot pepe, 1 links, 0 joints
Links:
- link 0: mass 3.642215640841591 -> 2.636581497308167; geometry collision cylinder length=1.9998 radius=0.6478170612570427; visual cylinder length=1.9998 radius=0.6478170612570427

File: midterm/part_b/source_code/my_code/test.urdf (robot description, URDF)
Before this commit: robot pepe, 6 links, 5 joints
Links:
- removed link 12
- removed link 13
- removed link 24
- added link 14, mass 1.5947442598778065; collision cylinder length=1.2315898695348884 radius=0.642003703675905; visual cylinder length=1.2315898695348884 radius=0.642003703675905
- added link 17, mass 1.5947442598778065; collision cylinder length=1.2315898695348884 radius=0.642003703675905; visual cylinder length=1.2315898695348884 radius=0.642003703675905
- added link 22, mass 1.5044046897544627; collision cylinder length=1.8868307141193543 radius=0.503780014280673; visual cylinder length=1.8868307141193543 radius=0.503780014280673
- added link 23, mass 1.5044046897544627; collision cylinder length=1.8868307141193543 radius=0.503780014280673; visual cylinder length=1.8868307141193543 radius=0.503780014280673
- added link 26, mass 1.5044046897544627; collision cylinder length=1.8868307141193543 radius=0.503780014280673; visual cylinder length=1.8868307141193543 radius=0.503780014280673
- added link 28, mass 1.5044046897544627; collision cylinder length=1.8868307141193543 radius=0.503780014280673; visual cylinder length=1.8868307141193543 radius=0.503780014280673
- added link 29, mass 1.5044046897544627; collision cylinder length=1.8868307141193543 radius=0.503780014280673; visual cylinder length=1.8868307141193543 radius=0.503780014280673
- link 0: mass 1.3201253554439543 -> 1.8854175460813747; geometry collision cylinder length=1.9998 radius=0.5478170612570428; visual cylinder length=1.9998 radius=0.5478170612570428
- link 11: mass 0.11181161068801812 -> 1.5947442598778065; geometry collision cylinder length=1.2315898695348884 radius=0.642003703675905; visual cylinder length=1.2315898695348884 radius=0.642003703675905
- link 25: mass 0.0005475799489116338 -> 1.5044046897544627; geometry collision cylinder length=1.8868307141193543 radius=0.503780014280673; visual cylinder length=1.8868307141193543 radius=0.503780014280673
Joints:
- removed joint 12_to_0
- removed joint 13_to_0
- removed joint 24_to_0
- removed joint 25_to_0
- added joint 14_to_0: type revolute, parent 0, child 14, origin xyz=0.4083539779659313 0.43078172763723277 0.1445608338794231 rpy=7.77085007801996 1.605921221101544 1.8170763717898664, axis 0 1 0, limit lower=3.1415 upper=-3.1415 effort=1 velocity=1
- added joint 17_to_0: type revolute, parent 0, child 17, origin xyz=0.4083539779659313 0.43078172763723277 0.1445608338794231 rpy=10.361133437359946 1.605921221101544 1.8170763717898664, axis 0 1 0, limit lower=3.1415 upper=-3.1415 effort=1 velocity=1
- added joint 22_to_11: type revolute, parent 11, child 22, origin xyz=0.5730807334560745 0.17423659666344593 0.4035162322813609 rpy=9.130658738083964 4.952894278360885 5.872512715142709, axis 1 0 0, limit lower=3.1415 upper=-3.1415 effort=1 velocity=1
- added joint 23_to_11: type revolute, parent 11, child 23, origin xyz=0.5730807334560745 0.17423659666344593 0.4035162322813609 rpy=13.695988107125945 4.952894278360885 5.872512715142709, axis 1 0 0, limit lower=3.1415 upper=-3.1415 effort=1 velocity=1
- added joint 25_to_14: type revolute, parent 14, child 25, origin xyz=0.5730807334560745 0.17423659666344593 0.4035162322813609 rpy=9.130658738083964 4.952894278360885 5.872512715142709, axis 1 0 0, limit lower=3.1415 upper=-3.1415 effort=1 velocity=1
- added joint 26_to_14: type revolute, parent 14, child 26, origin xyz=0.5730807334560745 0.17423659666344593 0.4035162322813609 rpy=13.695988107125945 4.952894278360885 5.872512715142709, axis 1 0 0, limit lower=3.1415 upper=-3.1415 effort=1 velocity=1
- added joint 28_to_17: type revolute, parent 17, child 28, origin xyz=0.5730807334560745 0.17423659666344593 0.4035162322813609 rpy=9.130658738083964 4.952894278360885 5.872512715142709, axis 1 0 0, limit lower=3.1415 upper=-3.1415 effort=1 velocity=1
- added joint 29_to_17: type revolute, parent 17, child 29, origin xyz=0.5730807334560745 0.17423659666344593 0.4035162322813609 rpy=13.695988107125945 4.952894278360885 5.872512715142709, axis 1 0 0, limit lower=3.1415 upper=-3.1415 effort=1 velocity=1
- joint 11_to_0: origin xyz=0.41559261142294956 0.1438599694240963 0.29914652633218375 rpy=5.537390934221668 2.4991748170154304 3.895525149863389 -> xyz=0.4083539779659313 0.43078172763723277 0.1445608338794231 rpy=5.180566718679973 1.605921221101544 1.8170763717898664

Commit message: Basic coursework pretty much done

File: midterm/part_b/source_code/my_code/temp0.urdf (robot description, URDF)
Before this commit: robot pepe, 1 links, 0 joints
Links:
- link 0: mass 2.636581497308167 -> 0.6387235666790397; geometry collision cylinder length=0.450587207684787 radius=0.6717259171243225; visual cylinder length=0.450587207684787 radius=0.6717259171243225
