Commit message: Start of changing of fitness

File: midterm/part_b/source_code/my_code/temp0.urdf (robot description, URDF)
Before this commit: robot pepe, 154 links, 153 joints
Links:
- removed link 1103
- removed link 152
- removed link 2104
- removed link 2129
- removed link 22
- removed link 227
- removed link 253
- removed link 278
- removed link 3105
- removed link 311
- removed link 3113
- removed link 3121
- removed link 3130
- removed link 3138
- removed link 3146
- removed link 319
- removed link 328
- removed link 33
- removed link 336
- removed link 344
- removed link 354
- removed link 362
- removed link 370
- removed link 379
- removed link 387
- removed link 395
- removed link 4106
- removed link 4114
- removed link 412
- removed link 4122
- removed link 4131
- removed link 4139
- removed link 4147
- removed link 420
- removed link 429
- removed link 437
- removed link 44
- removed link 445
- removed link 455
- removed link 463
- removed link 471
- removed link 480
- removed link 488
- removed link 496
- removed link 5101
- removed link 5107
- removed link 5109
- removed link 5111
- removed link 5115
- removed link 5117
- removed link 5119
- removed link 5123
- removed link 5125
- removed link 5127
- removed link 513
- removed link 5132
- removed link 5134
- removed link 5136
- removed link 5140
- removed link 5142
- removed link 5144
- removed link 5148
- removed link 515
- removed link 5150
- removed link 5152
- removed link 517
- removed link 521
- removed link 523
- removed link 525
- removed link 530
- removed link 532
- removed link 534
- removed link 538
- removed link 540
- removed link 542
- removed link 546
- removed link 548
- removed link 55
- removed link 550
- removed link 556
- removed link 558
- removed link 560
- removed link 564
- removed link 566
- removed link 568
- removed link 57
- removed link 572
- removed link 574
- removed link 576
- removed link 581
- removed link 583
- removed link 585
- removed link 589
- removed link 59
- removed link 591
- removed link 593
- removed link 597
- removed link 599
- removed link 610
- removed link 6100
- removed link 6102
- removed link 6108
- removed link 6110
- removed link 6112
- removed link 6116
- removed link 6118
- removed link 6120
- removed link 6124
- removed link 6126
- removed link 6128
- removed link 6133
- removed link 6135
- removed link 6137
- removed link 614
- removed link 6141
- removed link 6143
- removed link 6145
- removed link 6149
- removed link 6151
- removed link 6153
- removed link 616
- removed link 618
- removed link 622
- removed link 624
- removed link 626
- removed link 631
- removed link 633
- removed link 635
- removed link 639
- removed link 641
- removed link 643
- removed link 647
- removed link 649
- removed link 651
- removed link 657
- removed link 659
- removed link 66
- removed link 661
- removed link 665
- removed link 667
- removed link 669
- removed link 673
- removed link 675
- removed link 677
- removed link 68
- removed link 682
- removed link 684
- removed link 686
- removed link 690
- removed link 692
- removed link 694
- removed link 698
- added link 12, mass 1.480154782225108; collision cylinder length=0.4712421439808423 radius=0.9999; visual cylinder length=0.4712421439808423 radius=0.9999
- added link 13, mass 1.480154782225108; collision cylinder length=0.4712421439808423 radius=0.9999; visual cylinder length=0.4712421439808423 radius=0.9999
- link 0: mass 5.3728171262644695 -> 2.0798685134506556; geometry collision cylinder length=1.9998 radius=0.575373322585344; visual cylinder length=1.9998 radius=0.575373322585344
- link 11: mass 0.9233099306693617 -> 1.480154782225108; geometry collision cylinder length=0.4712421439808423 radius=0.9999; visual cylinder length=0.4712421439808423 radius=0.9999
Joints:
- removed joint 1103_to_0
- removed joint 152_to_0
- removed joint 2104_to_1103
- removed joint 2129_to_1103
- removed joint 227_to_11
- removed joint 22_to_11
- removed joint 253_to_152
- removed joint 278_to_152
- removed joint 3105_to_2104
- removed joint 3113_to_2104
- removed joint 311_to_22
- removed joint 3121_to_2104
- removed joint 3130_to_2129
- removed joint 3138_to_2129
- removed joint 3146_to_2129
- removed joint 319_to_22
- removed joint 328_to_227
- removed joint 336_to_227
- removed joint 33_to_22
- removed joint 344_to_227
- removed joint 354_to_253
- removed joint 362_to_253
- removed joint 370_to_253
- removed joint 379_to_278
- removed joint 387_to_278
- removed joint 395_to_278
- removed joint 4106_to_3105
- removed joint 4114_to_3113
- removed joint 4122_to_3121
- removed joint 412_to_311
- removed joint 4131_to_3130
- removed joint 4139_to_3138
- removed joint 4147_to_3146
- removed joint 420_to_319
- removed joint 429_to_328
- removed joint 437_to_336
- removed joint 445_to_344
- removed joint 44_to_33
- removed joint 455_to_354
- removed joint 463_to_362
- removed joint 471_to_370
- removed joint 480_to_379
- removed joint 488_to_387
- removed joint 496_to_395
- removed joint 5101_to_496
- removed joint 5107_to_4106
- removed joint 5109_to_4106
- removed joint 5111_to_4106
- removed joint 5115_to_4114
- removed joint 5117_to_4114
- removed joint 5119_to_4114
- removed joint 5123_to_4122
- removed joint 5125_to_4122
- removed joint 5127_to_4122
- removed joint 5132_to_4131
- removed joint 5134_to_4131
- removed joint 5136_to_4131
- removed joint 513_to_412
- removed joint 5140_to_4139
- removed joint 5142_to_4139
- removed joint 5144_to_4139
- removed joint 5148_to_4147
- removed joint 5150_to_4147
- removed joint 5152_to_4147
- removed joint 515_to_412
- removed joint 517_to_412
- removed joint 521_to_420
- removed joint 523_to_420
- removed joint 525_to_420
- removed joint 530_to_429
- removed joint 532_to_429
- removed joint 534_to_429
- removed joint 538_to_437
- removed joint 540_to_437
- removed joint 542_to_437
- removed joint 546_to_445
- removed joint 548_to_445
- removed joint 550_to_445
- removed joint 556_to_455
- removed joint 558_to_455
- removed joint 55_to_44
- removed joint 560_to_455
- removed joint 564_to_463
- removed joint 566_to_463
- removed joint 568_to_463
- removed joint 572_to_471
- removed joint 574_to_471
- removed joint 576_to_471
- removed joint 57_to_44
- removed joint 581_to_480
- removed joint 583_to_480
- removed joint 585_to_480
- removed joint 589_to_488
- removed joint 591_to_488
- removed joint 593_to_488
- removed joint 597_to_496
- removed joint 599_to_496
- removed joint 59_to_44
- removed joint 6100_to_599
- removed joint 6102_to_5101
- removed joint 6108_to_5107
- removed joint 610_to_59
- removed joint 6110_to_5109
- removed joint 6112_to_5111
- removed joint 6116_to_5115
- removed joint 6118_to_5117
- removed joint 6120_to_5119
- removed joint 6124_to_5123
- removed joint 6126_to_5125
- removed joint 6128_to_5127
- removed joint 6133_to_5132
- removed joint 6135_to_5134
- removed joint 6137_to_5136
- removed joint 6141_to_5140
- removed joint 6143_to_5142
- removed joint 6145_to_5144
- removed joint 6149_to_5148
- removed joint 614_to_513
- removed joint 6151_to_5150
- removed joint 6153_to_5152
- removed joint 616_to_515
- removed joint 618_to_517
- removed joint 622_to_521
- removed joint 624_to_523
- removed joint 626_to_525
- removed joint 631_to_530
- removed joint 633_to_532
- removed joint 635_to_534
- removed joint 639_to_538
- removed joint 641_to_540
- removed joint 643_to_542
- removed joint 647_to_546
- removed joint 649_to_548
- removed joint 651_to_550
- removed joint 657_to_556
- removed joint 659_to_558
- removed joint 661_to_560
- removed joint 665_to_564
- removed joint 667_to_566
- removed joint 669_to_568
- removed joint 66_to_55
- removed joint 673_to_572
- removed joint 675_to_574
- removed joint 677_to_576
- removed joint 682_to_581
- removed joint 684_to_583
- removed joint 686_to_585
- removed joint 68_to_57
- removed joint 690_to_589
- removed joint 692_to_591
- removed joint 694_to_593
- removed joint 698_to_597
- added joint 12_to_0: type revolute, parent 0, child 12, origin xyz=0.9620143527404951 0.9992085664588672 0.5231248412405833 rpy=18.847670965946605 6.282556988648868 6.282556988648868, axis 0 0 1, limit lower=3.1415 upper=-3.1415 effort=1 velocity=1
- added joint 13_to_0: type revolute, parent 0, child 13, origin xyz=0.9620143527404951 0.9992085664588672 0.5231248412405833 rpy=25.130227954595473 6.282556988648868 6.282556988648868, axis 0 0 1, limit lower=3.1415 upper=-3.1415 effort=1 velocity=1
- joint 11_to_0: axis 0 1 0 -> 0 0 1; origin xyz=0.8496673682276968 0.23520769677330514 0.326170469526187 rpy=10.808392987238653 6.282556988648868 0.5422677742866492 -> xyz=0.9620143527404951 0.9992085664588672 0.5231248412405833 rpy=12.565113977297736 6.282556988648868 6.282556988648868

File: midterm/part_b/source_code/my_code/test.urdf (robot description, URDF)
Before this commit: robot pepe, 16 links, 15 joints
Links:
- removed link 111
- removed link 16
- removed link 212
- removed link 213
- removed link 214
- removed link 22
- removed link 23
- removed link 24
- removed link 27
- removed link 28
- removed link 29
- removed link 310
- removed link 315
- removed link 35
- added link 12, mass 2.0798685134506556; collision cylinder length=1.9998 radius=0.575373322585344; visual cylinder length=1.9998 radius=0.575373322585344
- added link 13, mass 2.0798685134506556; collision cylinder length=1.9998 radius=0.575373322585344; visual cylinder length=1.9998 radius=0.575373322585344
- link 0: mass 6.281300540076709 -> 1.480154782225108; geometry collision cylinder length=0.4712421439808423 radius=0.9999; visual cylinder length=0.4712421439808423 radius=0.9999
- link 11: mass 6.281300540076709 -> 2.0798685134506556; geometry collision cylinder length=1.9998 radius=0.575373322585344; visual cylinder length=1.9998 radius=0.575373322585344
Joints:
- removed joint 111_to_0
- removed joint 16_to_0
- removed joint 212_to_111
- removed joint 213_to_111
- removed joint 214_to_111
- removed joint 22_to_11
- removed joint 23_to_11
- removed joint 24_to_11
- removed joint 27_to_16
- removed joint 28_to_16
- removed joint 29_to_16
- removed joint 310_to_16
- removed joint 315_to_111
- removed joint 35_to_11
- added joint 12_to_0: type revolute, parent 0, child 12, origin xyz=0.5589244085207674 0.43366660064400775 0.6045531313245386 rpy=15.626529090902476 0.6822935711469509 4.514231444512896, axis 0 1 0, limit lower=3.1415 upper=-3.1415 effort=1 velocity=1
- added joint 13_to_0: type revolute, parent 0, child 13, origin xyz=0.5589244085207674 0.43366660064400775 0.6045531313245386 rpy=20.835372121203303 0.6822935711469509 4.514231444512896, axis 0 1 0, limit lower=3.1415 upper=-3.1415 effort=1 velocity=1
- joint 11_to_0: axis 0 0 1 -> 0 1 0; origin xyz=0.9999 0.9999 0.9999 rpy=11.500418621995479 6.282556988648868 6.121241751000677 -> xyz=0.5589244085207674 0.43366660064400775 0.6045531313245386 rpy=10.417686060601651 0.6822935711469509 4.514231444512896
