Commit message: Work on project

File: midterm/part_b/source_code/my_code/temp0.urdf (robot description, URDF)
Before this commit: robot pepe, 4 links, 3 joints
Links:
- removed link 12
- removed link 13
- added link 110, mass 1.358954566976295; collision cylinder length=1.9998 radius=0.46508705353763646; visual cylinder length=1.9998 radius=0.46508705353763646
- added link 211, mass 1.358954566976295; collision cylinder length=1.9998 radius=0.46508705353763646; visual cylinder length=1.9998 radius=0.46508705353763646
- added link 215, mass 1.358954566976295; collision cylinder length=1.9998 radius=0.46508705353763646; visual cylinder length=1.9998 radius=0.46508705353763646
- added link 22, mass 1.358954566976295; collision cylinder length=1.9998 radius=0.46508705353763646; visual cylinder length=1.9998 radius=0.46508705353763646
- added link 26, mass 1.358954566976295; collision cylinder length=1.9998 radius=0.46508705353763646; visual cylinder length=1.9998 radius=0.46508705353763646
- added link 312, mass 4.61871276772004; collision cylinder length=1.4732178765428487 radius=0.9989690911035517; visual cylinder length=1.4732178765428487 radius=0.9989690911035517
- added link 313, mass 4.61871276772004; collision cylinder length=1.4732178765428487 radius=0.9989690911035517; visual cylinder length=1.4732178765428487 radius=0.9989690911035517
- added link 314, mass 4.61871276772004; collision cylinder length=1.4732178765428487 radius=0.9989690911035517; visual cylinder length=1.4732178765428487 radius=0.9989690911035517
- added link 316, mass 4.61871276772004; collision cylinder length=1.4732178765428487 radius=0.9989690911035517; visual cylinder length=1.4732178765428487 radius=0.9989690911035517
- added link 317, mass 4.61871276772004; collision cylinder length=1.4732178765428487 radius=0.9989690911035517; visual cylinder length=1.4732178765428487 radius=0.9989690911035517
- added link 318, mass 4.61871276772004; collision cylinder length=1.4732178765428487 radius=0.9989690911035517; visual cylinder length=1.4732178765428487 radius=0.9989690911035517
- added link 33, mass 4.61871276772004; collision cylinder length=1.4732178765428487 radius=0.9989690911035517; visual cylinder length=1.4732178765428487 radius=0.9989690911035517
- added link 34, mass 4.61871276772004; collision cylinder length=1.4732178765428487 radius=0.9989690911035517; visual cylinder length=1.4732178765428487 radius=0.9989690911035517
- added link 35, mass 4.61871276772004; collision cylinder length=1.4732178765428487 radius=0.9989690911035517; visual cylinder length=1.4732178765428487 radius=0.9989690911035517
- added link 37, mass 4.61871276772004; collision cylinder length=1.4732178765428487 radius=0.9989690911035517; visual cylinder length=1.4732178765428487 radius=0.9989690911035517
- added link 38, mass 4.61871276772004; collision cylinder length=1.4732178765428487 radius=0.9989690911035517; visual cylinder length=1.4732178765428487 radius=0.9989690911035517
- added link 39, mass 4.61871276772004; collision cylinder length=1.4732178765428487 radius=0.9989690911035517; visual cylinder length=1.4732178765428487 radius=0.9989690911035517
- link 0: mass 2.0798685134506556 -> 4.61871276772004; geometry collision cylinder length=1.4732178765428487 radius=0.9989690911035517; visual cylinder length=1.4732178765428487 radius=0.9989690911035517
- link 11: mass 1.480154782225108 -> 1.358954566976295; geometry collision cylinder length=1.9998 radius=0.46508705353763646; visual cylinder length=1.9998 radius=0.46508705353763646
Joints:
- removed joint 12_to_0
- removed joint 13_to_0
- added joint 110_to_0: type revolute, parent 0, child 110, origin xyz=0.9738900462936835 0.8229201595427645 0.880726920477414 rpy=18.620643149996486 4.396687861377438 2.571183777630715, axis 0 0 1, limit lower=3.1415 upper=-3.1415 effort=1 velocity=1
- added joint 211_to_110: type revolute, parent 110, child 211, origin xyz=0.9999 0.7229201595427646 0.880726920477414 rpy=11.157125038561741 4.396687861377438 2.571183777630715, axis 0 0 1, limit lower=3.1415 upper=-3.1415 effort=1 velocity=1
- added joint 215_to_110: type revolute, parent 110, child 215, origin xyz=0.9999 0.7229201595427646 0.880726920477414 rpy=16.73568755784261 4.396687861377438 2.571183777630715, axis 0 0 1, limit lower=3.1415 upper=-3.1415 effort=1 velocity=1
- added joint 22_to_11: type revolute, parent 11, child 22, origin xyz=0.9999 0.7229201595427646 0.880726920477414 rpy=11.157125038561741 4.396687861377438 2.571183777630715, axis 0 0 1, limit lower=3.1415 upper=-3.1415 effort=1 velocity=1
- added joint 26_to_11: type revolute, parent 11, child 26, origin xyz=0.9999 0.7229201595427646 0.880726920477414 rpy=16.73568755784261 4.396687861377438 2.571183777630715, axis 0 0 1, limit lower=3.1415 upper=-3.1415 effort=1 velocity=1
- added joint 312_to_211: type revolute, parent 211, child 312, origin xyz=0.4262248606372623 0.8198653371329021 0.15807976346402933 rpy=9.378985428131854 1.500870120141237 2.8933777920457926, axis 0 1 0, limit lower=3.1415 upper=-3.1415 effort=1 velocity=1
- added joint 313_to_211: type revolute, parent 211, child 313, origin xyz=0.4262248606372623 0.8198653371329021 0.15807976346402933 rpy=14.06847814219778 1.500870120141237 2.8933777920457926, axis 0 1 0, limit lower=3.1415 upper=-3.1415 effort=1 velocity=1
- added joint 314_to_211: type revolute, parent 211, child 314, origin xyz=0.4262248606372623 0.8198653371329021 0.15807976346402933 rpy=18.757970856263707 1.500870120141237 2.8933777920457926, axis 0 1 0, limit lower=3.1415 upper=-3.1415 effort=1 velocity=1
- added joint 316_to_215: type revolute, parent 215, child 316, origin xyz=0.4262248606372623 0.8198653371329021 0.15807976346402933 rpy=9.378985428131854 1.500870120141237 2.8933777920457926, axis 0 1 0, limit lower=3.1415 upper=-3.1415 effort=1 velocity=1
- added joint 317_to_215: type revolute, parent 215, child 317, origin xyz=0.4262248606372623 0.8198653371329021 0.15807976346402933 rpy=14.06847814219778 1.500870120141237 2.8933777920457926, axis 0 1 0, limit lower=3.1415 upper=-3.1415 effort=1 velocity=1
- added joint 318_to_215: type revolute, parent 215, child 318, origin xyz=0.4262248606372623 0.8198653371329021 0.15807976346402933 rpy=18.757970856263707 1.500870120141237 2.8933777920457926, axis 0 1 0, limit lower=3.1415 upper=-3.1415 effort=1 velocity=1
- added joint 33_to_22: type revolute, parent 22, child 33, origin xyz=0.4262248606372623 0.8198653371329021 0.15807976346402933 rpy=9.378985428131854 1.500870120141237 2.8933777920457926, axis 0 1 0, limit lower=3.1415 upper=-3.1415 effort=1 velocity=1
- added joint 34_to_22: type revolute, parent 22, child 34, origin xyz=0.4262248606372623 0.8198653371329021 0.15807976346402933 rpy=14.06847814219778 1.500870120141237 2.8933777920457926, axis 0 1 0, limit lower=3.1415 upper=-3.1415 effort=1 velocity=1
- added joint 35_to_22: type revolute, parent 22, child 35, origin xyz=0.4262248606372623 0.8198653371329021 0.15807976346402933 rpy=18.757970856263707 1.500870120141237 2.8933777920457926, axis 0 1 0, limit lower=3.1415 upper=-3.1415 effort=1 velocity=1
- added joint 37_to_26: type revolute, parent 26, child 37, origin xyz=0.4262248606372623 0.8198653371329021 0.15807976346402933 rpy=9.378985428131854 1.500870120141237 2.8933777920457926, axis 0 1 0, limit lower=3.1415 upper=-3.1415 effort=1 velocity=1
- added joint 38_to_26: type revolute, parent 26, child 38, origin xyz=0.4262248606372623 0.8198653371329021 0.15807976346402933 rpy=14.06847814219778 1.500870120141237 2.8933777920457926, axis 0 1 0, limit lower=3.1415 upper=-3.1415 effort=1 velocity=1
- added joint 39_to_26: type revolute, parent 26, child 39, origin xyz=0.4262248606372623 0.8198653371329021 0.15807976346402933 rpy=18.757970856263707 1.500870120141237 2.8933777920457926, axis 0 1 0, limit lower=3.1415 upper=-3.1415 effort=1 velocity=1
- joint 11_to_0: origin xyz=0.9620143527404951 0.9992085664588672 0.5231248412405833 rpy=12.565113977297736 6.282556988648868 6.282556988648868 -> xyz=0.9738900462936835 0.8229201595427645 0.880726920477414 rpy=12.413762099997657 4.396687861377438 2.571183777630715

File: midterm/part_b/source_code/my_code/test.urdf (robot description, URDF)
Before this commit: robot pepe, 4 links, 3 joints
Links:
- removed link 12
- removed link 13
- added link 18, mass 2.006167320569381; collision cylinder length=1.9998 radius=0.5650870535376364; visual cylinder length=1.9998 radius=0.5650870535376364
- added link 210, mass 4.134239237027495; collision cylinder length=1.3162324543233237 radius=0.9999; visual cylinder length=1.3162324543233237 radius=0.9999
- added link 211, mass 4.134239237027495; collision cylinder length=1.3162324543233237 radius=0.9999; visual cylinder length=1.3162324543233237 radius=0.9999
- added link 22, mass 4.134239237027495; collision cylinder length=1.3162324543233237 radius=0.9999; visual cylinder length=1.3162324543233237 radius=0.9999
- added link 23, mass 4.134239237027495; collision cylinder length=1.3162324543233237 radius=0.9999; visual cylinder length=1.3162324543233237 radius=0.9999
- added link 24, mass 4.134239237027495; collision cylinder length=1.3162324543233237 radius=0.9999; visual cylinder length=1.3162324543233237 radius=0.9999
- added link 29, mass 4.134239237027495; collision cylinder length=1.3162324543233237 radius=0.9999; visual cylinder length=1.3162324543233237 radius=0.9999
- added link 312, mass 0.10972924231903197; collision cylinder length=0.3810548072120239 radius=0.30275584154777135; visual cylinder length=0.3810548072120239 radius=0.30275584154777135
- added link 313, mass 0.10972924231903197; collision cylinder length=0.3810548072120239 radius=0.30275584154777135; visual cylinder length=0.3810548072120239 radius=0.30275584154777135
- added link 314, mass 0.10972924231903197; collision cylinder length=0.3810548072120239 radius=0.30275584154777135; visual cylinder length=0.3810548072120239 radius=0.30275584154777135
- added link 35, mass 0.10972924231903197; collision cylinder length=0.3810548072120239 radius=0.30275584154777135; visual cylinder length=0.3810548072120239 radius=0.30275584154777135
- added link 36, mass 0.10972924231903197; collision cylinder length=0.3810548072120239 radius=0.30275584154777135; visual cylinder length=0.3810548072120239 radius=0.30275584154777135
- added link 37, mass 0.10972924231903197; collision cylinder length=0.3810548072120239 radius=0.30275584154777135; visual cylinder length=0.3810548072120239 radius=0.30275584154777135
- link 0: mass 1.480154782225108 -> 1.358954566976295; geometry collision cylinder length=1.9998 radius=0.46508705353763646; visual cylinder length=1.9998 radius=0.46508705353763646
- link 11: mass 2.0798685134506556 -> 2.006167320569381; geometry collision cylinder length=1.9998 radius=0.5650870535376364; visual cylinder length=1.9998 radius=0.5650870535376364
Joints:
- removed joint 12_to_0
- removed joint 13_to_0
- added joint 18_to_0: type revolute, parent 0, child 18, origin xyz=0.9999 0.7229201595427646 0.880726920477414 rpy=16.73568755784261 3.768369330659479 1.9428652469127565, axis 0 0 1, limit lower=3.1415 upper=-3.1415 effort=1 velocity=1
- added joint 210_to_18: type revolute, parent 18, child 210, origin xyz=0.5820242690305131 0.6987132297414442 0.6222414845175622 rpy=11.590534429516348 2.676780437967274 3.5813951072728796, axis 0 0 1, limit lower=3.1415 upper=-3.1415 effort=1 velocity=1
- added joint 211_to_18: type revolute, parent 18, child 211, origin xyz=0.5820242690305131 0.6987132297414442 0.6222414845175622 rpy=15.454045906021797 2.676780437967274 3.5813951072728796, axis 0 0 1, limit lower=3.1415 upper=-3.1415 effort=1 velocity=1
- added joint 22_to_11: type revolute, parent 11, child 22, origin xyz=0.5820242690305131 0.6987132297414442 0.6222414845175622 rpy=7.7270229530108985 2.676780437967274 3.5813951072728796, axis 0 0 1, limit lower=3.1415 upper=-3.1415 effort=1 velocity=1
- added joint 23_to_11: type revolute, parent 11, child 23, origin xyz=0.5820242690305131 0.6987132297414442 0.6222414845175622 rpy=11.590534429516348 2.676780437967274 3.5813951072728796, axis 0 0 1, limit lower=3.1415 upper=-3.1415 effort=1 velocity=1
- added joint 24_to_11: type revolute, parent 11, child 24, origin xyz=0.5820242690305131 0.6987132297414442 0.6222414845175622 rpy=15.454045906021797 2.676780437967274 3.5813951072728796, axis 0 0 1, limit lower=3.1415 upper=-3.1415 effort=1 velocity=1
- added joint 29_to_18: type revolute, parent 18, child 29, origin xyz=0.5820242690305131 0.6987132297414442 0.6222414845175622 rpy=7.7270229530108985 2.676780437967274 3.5813951072728796, axis 0 0 1, limit lower=3.1415 upper=-3.1415 effort=1 velocity=1
- added joint 312_to_18: type revolute, parent 18, child 312, origin xyz=0.012436390198700797 0.43411320039596357 0.15358209544850143 rpy=4.434879981566325 3.8278787320810093 0.08186299012965713, axis 0 0 1, limit lower=3.1415 upper=-3.1415 effort=1 velocity=1
- added joint 313_to_18: type revolute, parent 18, child 313, origin xyz=0.012436390198700797 0.43411320039596357 0.15358209544850143 rpy=5.32185597787959 3.8278787320810093 0.08186299012965713, axis 0 0 1, limit lower=3.1415 upper=-3.1415 effort=1 velocity=1
- added joint 314_to_18: type revolute, parent 18, child 314, origin xyz=0.012436390198700797 0.43411320039596357 0.15358209544850143 rpy=6.208831974192854 3.8278787320810093 0.08186299012965713, axis 0 0 1, limit lower=3.1415 upper=-3.1415 effort=1 velocity=1
- added joint 35_to_11: type revolute, parent 11, child 35, origin xyz=0.012436390198700797 0.43411320039596357 0.15358209544850143 rpy=4.434879981566325 3.8278787320810093 0.08186299012965713, axis 0 0 1, limit lower=3.1415 upper=-3.1415 effort=1 velocity=1
- added joint 36_to_11: type revolute, parent 11, child 36, origin xyz=0.012436390198700797 0.43411320039596357 0.15358209544850143 rpy=5.32185597787959 3.8278787320810093 0.08186299012965713, axis 0 0 1, limit lower=3.1415 upper=-3.1415 effort=1 velocity=1
- added joint 37_to_11: type revolute, parent 11, child 37, origin xyz=0.012436390198700797 0.43411320039596357 0.15358209544850143 rpy=6.208831974192854 3.8278787320810093 0.08186299012965713, axis 0 0 1, limit lower=3.1415 upper=-3.1415 effort=1 velocity=1
- joint 11_to_0: axis 0 1 0 -> 0 0 1; origin xyz=0.5589244085207674 0.43366660064400775 0.6045531313245386 rpy=10.417686060601651 0.6822935711469509 4.514231444512896 -> xyz=0.9999 0.7229201595427646 0.880726920477414 rpy=11.157125038561741 3.768369330659479 1.9428652469127565

Commit message: Work on project

File: midterm/part_b/source_code/my_code/temp0.urdf (robot description, URDF)
Before this commit: robot pepe, 19 links, 18 joints
Links:
- removed link 11
- removed link 110
- removed link 211
- removed link 215
- removed link 22
- removed link 26
- removed link 312
- removed link 313
- removed link 314
- removed link 316
- removed link 317
- removed link 318
- removed link 33
- removed link 34
- removed link 35
- removed link 37
- removed link 38
- removed link 39
- link 0: mass 4.61871276772004 -> 3.0943477562768655; geometry collision cylinder length=1.1511851219191618 radius=0.9249900042171386; visual cylinder length=1.1511851219191618 radius=0.9249900042171386
Joints:
- removed joint 110_to_0
- removed joint 11_to_0
- removed joint 211_to_110
- removed joint 215_to_110
- removed joint 22_to_11
- removed joint 26_to_11
- removed joint 312_to_211
- removed joint 313_to_211
- removed joint 314_to_211
- removed joint 316_to_215
- removed joint 317_to_215
- removed joint 318_to_215
- removed joint 33_to_22
- removed joint 34_to_22
- removed joint 35_to_22
- removed joint 37_to_26
- removed joint 38_to_26
- removed joint 39_to_26

File: midterm/part_b/source_code/my_code/test.urdf (robot description, URDF)
Before this commit: robot pepe, 15 links, 14 joints
Links:
- removed link 18
- removed link 210
- removed link 211
- removed link 29
- removed link 312
- removed link 313
- removed link 314
- removed link 35
- removed link 36
- removed link 37
- link 0: mass 1.358954566976295 -> 2.5930331903046304; geometry collision cylinder length=1.9998 radius=0.6424448018084249; visual cylinder length=1.9998 radius=0.6424448018084249
- link 11: mass 2.006167320569381 -> 0.358686335824467; geometry collision cylinder length=1.450153021574419 radius=0.2805921804913516; visual cylinder length=1.450153021574419 radius=0.2805921804913516
- link 22: mass 4.134239237027495 -> 6.281300540076709; geometry collision cylinder length=1.9998 radius=0.9999; visual cylinder length=1.9998 radius=0.9999
- link 23: mass 4.134239237027495 -> 6.281300540076709; geometry collision cylinder length=1.9998 radius=0.9999; visual cylinder length=1.9998 radius=0.9999
- link 24: mass 4.134239237027495 -> 6.281300540076709; geometry collision cylinder length=1.9998 radius=0.9999; visual cylinder length=1.9998 radius=0.9999
Joints:
- removed joint 18_to_0
- removed joint 210_to_18
- removed joint 211_to_18
- removed joint 29_to_18
- removed joint 312_to_18
- removed joint 313_to_18
- removed joint 314_to_18
- removed joint 35_to_11
- removed joint 36_to_11
- removed joint 37_to_11
- joint 11_to_0: axis 0 0 1 -> 1 0 0; origin xyz=0.9999 0.7229201595427646 0.880726920477414 rpy=11.157125038561741 3.768369330659479 1.9428652469127565 -> xyz=0.3460188446689044 0.6833411772002934 0.7033764135855681 rpy=9.077885448262554 1.0902438349063948 0.6867123107155225
- joint 22_to_11: origin xyz=0.5820242690305131 0.6987132297414442 0.6222414845175622 rpy=7.7270229530108985 2.676780437967274 3.5813951072728796 -> xyz=0.45405508768181935 0.892176459734454 0.9999 rpy=8.66565279580873 3.5976894662525485 2.1261173357679928
- joint 23_to_11: origin xyz=0.5820242690305131 0.6987132297414442 0.6222414845175622 rpy=11.590534429516348 2.676780437967274 3.5813951072728796 -> xyz=0.45405508768181935 0.892176459734454 0.9999 rpy=12.998479193713095 3.5976894662525485 2.1261173357679928
- joint 24_to_11: origin xyz=0.5820242690305131 0.6987132297414442 0.6222414845175622 rpy=15.454045906021797 2.676780437967274 3.5813951072728796 -> xyz=0.45405508768181935 0.892176459734454 0.9999 rpy=17.33130559161746 3.5976894662525485 2.1261173357679928
