Commit message: WOrk on project

File: midterm/part_b/source_code/my_code/temp0.urdf (robot description, URDF)
Before this commit: robot pepe, 1 links, 0 joints
Links:
- added link 11, mass 6.0568130706387295; collision cylinder length=1.928329125693357 radius=0.9999; visual cylinder length=1.928329125693357 radius=0.9999
- added link 114, mass 6.0568130706387295; collision cylinder length=1.928329125693357 radius=0.9999; visual cylinder length=1.928329125693357 radius=0.9999
- added link 127, mass 6.0568130706387295; collision cylinder length=1.928329125693357 radius=0.9999; visual cylinder length=1.928329125693357 radius=0.9999
- added link 210, mass 6.0568130706387295; collision cylinder length=1.928329125693357 radius=0.9999; visual cylinder length=1.928329125693357 radius=0.9999
- added link 215, mass 6.0568130706387295; collision cylinder length=1.928329125693357 radius=0.9999; visual cylinder length=1.928329125693357 radius=0.9999
- added link 219, mass 6.0568130706387295; collision cylinder length=1.928329125693357 radius=0.9999; visual cylinder length=1.928329125693357 radius=0.9999
- added link 22, mass 6.0568130706387295; collision cylinder length=1.928329125693357 radius=0.9999; visual cylinder length=1.928329125693357 radius=0.9999
- added link 223, mass 6.0568130706387295; collision cylinder length=1.928329125693357 radius=0.9999; visual cylinder length=1.928329125693357 radius=0.9999
- added link 228, mass 6.0568130706387295; collision cylinder length=1.928329125693357 radius=0.9999; visual cylinder length=1.928329125693357 radius=0.9999
- added link 232, mass 6.0568130706387295; collision cylinder length=1.928329125693357 radius=0.9999; visual cylinder length=1.928329125693357 radius=0.9999
- added link 236, mass 6.0568130706387295; collision cylinder length=1.928329125693357 radius=0.9999; visual cylinder length=1.928329125693357 radius=0.9999
- added link 26, mass 6.0568130706387295; collision cylinder length=1.928329125693357 radius=0.9999; visual cylinder length=1.928329125693357 radius=0.9999
- added link 311, mass 6.0568130706387295; collision cylinder length=1.928329125693357 radius=0.9999; visual cylinder length=1.928329125693357 radius=0.9999
- added link 312, mass 6.0568130706387295; collision cylinder length=1.928329125693357 radius=0.9999; visual cylinder length=1.928329125693357 radius=0.9999
- added link 313, mass 6.0568130706387295; collision cylinder length=1.928329125693357 radius=0.9999; visual cylinder length=1.928329125693357 radius=0.9999
- added link 316, mass 6.0568130706387295; collision cylinder length=1.928329125693357 radius=0.9999; visual cylinder length=1.928329125693357 radius=0.9999
- added link 317, mass 6.0568130706387295; collision cylinder length=1.928329125693357 radius=0.9999; visual cylinder length=1.928329125693357 radius=0.9999
- added link 318, mass 6.0568130706387295; collision cylinder length=1.928329125693357 radius=0.9999; visual cylinder length=1.928329125693357 radius=0.9999
- added link 320, mass 6.0568130706387295; collision cylinder length=1.928329125693357 radius=0.9999; visual cylinder length=1.928329125693357 radius=0.9999
- added link 321, mass 6.0568130706387295; collision cylinder length=1.928329125693357 radius=0.9999; visual cylinder length=1.928329125693357 radius=0.9999
- added link 322, mass 6.0568130706387295; collision cylinder length=1.928329125693357 radius=0.9999; visual cylinder length=1.928329125693357 radius=0.9999
- added link 324, mass 6.0568130706387295; collision cylinder length=1.928329125693357 radius=0.9999; visual cylinder length=1.928329125693357 radius=0.9999
- added link 325, mass 6.0568130706387295; collision cylinder length=1.928329125693357 radius=0.9999; visual cylinder length=1.928329125693357 radius=0.9999
- added link 326, mass 6.0568130706387295; collision cylinder length=1.928329125693357 radius=0.9999; visual cylinder length=1.928329125693357 radius=0.9999
- added link 329, mass 6.0568130706387295; collision cylinder length=1.928329125693357 radius=0.9999; visual cylinder length=1.928329125693357 radius=0.9999
- added link 33, mass 6.0568130706387295; collision cylinder length=1.928329125693357 radius=0.9999; visual cylinder length=1.928329125693357 radius=0.9999
- added link 330, mass 6.0568130706387295; collision cylinder length=1.928329125693357 radius=0.9999; visual cylinder length=1.928329125693357 radius=0.9999
- added link 331, mass 6.0568130706387295; collision cylinder length=1.928329125693357 radius=0.9999; visual cylinder length=1.928329125693357 radius=0.9999
- added link 333, mass 6.0568130706387295; collision cylinder length=1.928329125693357 radius=0.9999; visual cylinder length=1.928329125693357 radius=0.9999
- added link 334, mass 6.0568130706387295; collision cylinder length=1.928329125693357 radius=0.9999; visual cylinder length=1.928329125693357 radius=0.9999
- added link 335, mass 6.0568130706387295; collision cylinder length=1.928329125693357 radius=0.9999; visual cylinder length=1.928329125693357 radius=0.9999
- added link 337, mass 6.0568130706387295; collision cylinder length=1.928329125693357 radius=0.9999; visual cylinder length=1.928329125693357 radius=0.9999
- added link 338, mass 6.0568130706387295; collision cylinder length=1.928329125693357 radius=0.9999; visual cylinder length=1.928329125693357 radius=0.9999
- added link 339, mass 6.0568130706387295; collision cylinder length=1.928329125693357 radius=0.9999; visual cylinder length=1.928329125693357 radius=0.9999
- added link 34, mass 6.0568130706387295; collision cylinder length=1.928329125693357 radius=0.9999; visual cylinder length=1.928329125693357 radius=0.9999
- added link 35, mass 6.0568130706387295; collision cylinder length=1.928329125693357 radius=0.9999; visual cylinder length=1.928329125693357 radius=0.9999
- added link 37, mass 6.0568130706387295; collision cylinder length=1.928329125693357 radius=0.9999; visual cylinder length=1.928329125693357 radius=0.9999
- added link 38, mass 6.0568130706387295; collision cylinder length=1.928329125693357 radius=0.9999; visual cylinder length=1.928329125693357 radius=0.9999
- added link 39, mass 6.0568130706387295; collision cylinder length=1.928329125693357 radius=0.9999; visual cylinder length=1.928329125693357 radius=0.9999
- link 0: mass 3.0943477562768655 -> 0.16089181704610028; geometry collision cylinder length=1.121906487419306 radius=0.21365532050541058; visual cylinder length=1.121906487419306 radius=0.21365532050541058
Joints:
- added joint 114_to_0: type revolute, parent 0, child 114, origin xyz=0.9999 0.3535889622219287 0.9606944566278526 rpy=16.911555307260638 6.282556988648868 6.0958890871509315, axis 1 0 0, limit lower=3.1415 upper=-3.1415 effort=1 velocity=1
- added joint 11_to_0: type revolute, parent 0, child 11, origin xyz=0.9999 0.3535889622219287 0.9606944566278526 rpy=11.274370204840425 6.282556988648868 6.0958890871509315, axis 1 0 0, limit lower=3.1415 upper=-3.1415 effort=1 velocity=1
- added joint 127_to_0: type revolute, parent 0, child 127, origin xyz=0.9999 0.3535889622219287 0.9606944566278526 rpy=22.54874040968085 6.282556988648868 6.0958890871509315, axis 1 0 0, limit lower=3.1415 upper=-3.1415 effort=1 velocity=1
- added joint 210_to_11: type revolute, parent 11, child 210, origin xyz=0.864255060277676 0.7535889622219286 0.8606944566278526 rpy=20.035466286809015 5.356506984867917 6.0958890871509315, axis 1 0 0, limit lower=3.1415 upper=-3.1415 effort=1 velocity=1
- added joint 215_to_114: type revolute, parent 114, child 215, origin xyz=0.864255060277676 0.7535889622219286 0.8606944566278526 rpy=10.017733143404508 5.356506984867917 6.0958890871509315, axis 1 0 0, limit lower=3.1415 upper=-3.1415 effort=1 velocity=1
- added joint 219_to_114: type revolute, parent 114, child 219, origin xyz=0.864255060277676 0.7535889622219286 0.8606944566278526 rpy=15.026599715106762 5.356506984867917 6.0958890871509315, axis 1 0 0, limit lower=3.1415 upper=-3.1415 effort=1 velocity=1
- added joint 223_to_114: type revolute, parent 114, child 223, origin xyz=0.864255060277676 0.7535889622219286 0.8606944566278526 rpy=20.035466286809015 5.356506984867917 6.0958890871509315, axis 1 0 0, limit lower=3.1415 upper=-3.1415 effort=1 velocity=1
- added joint 228_to_127: type revolute, parent 127, child 228, origin xyz=0.864255060277676 0.7535889622219286 0.8606944566278526 rpy=10.017733143404508 5.356506984867917 6.0958890871509315, axis 1 0 0, limit lower=3.1415 upper=-3.1415 effort=1 velocity=1
- added joint 22_to_11: type revolute, parent 11, child 22, origin xyz=0.864255060277676 0.7535889622219286 0.8606944566278526 rpy=10.017733143404508 5.356506984867917 6.0958890871509315, axis 1 0 0, limit lower=3.1415 upper=-3.1415 effort=1 velocity=1
- added joint 232_to_127: type revolute, parent 127, child 232, origin xyz=0.864255060277676 0.7535889622219286 0.8606944566278526 rpy=15.026599715106762 5.356506984867917 6.0958890871509315, axis 1 0 0, limit lower=3.1415 upper=-3.1415 effort=1 velocity=1
- added joint 236_to_127: type revolute, parent 127, child 236, origin xyz=0.864255060277676 0.7535889622219286 0.8606944566278526 rpy=20.035466286809015 5.356506984867917 6.0958890871509315, axis 1 0 0, limit lower=3.1415 upper=-3.1415 effort=1 velocity=1
- added joint 26_to_11: type revolute, parent 11, child 26, origin xyz=0.864255060277676 0.7535889622219286 0.8606944566278526 rpy=15.026599715106762 5.356506984867917 6.0958890871509315, axis 1 0 0, limit lower=3.1415 upper=-3.1415 effort=1 velocity=1
- added joint 311_to_210: type revolute, parent 210, child 311, origin xyz=0.9999 0.4535889622219287 0.8606944566278526 rpy=12.53100726627634 6.282556988648868 6.0958890871509315, axis 1 0 0, limit lower=3.1415 upper=-3.1415 effort=1 velocity=1
- added joint 312_to_210: type revolute, parent 210, child 312, origin xyz=0.9999 0.4535889622219287 0.8606944566278526 rpy=18.79651089941451 6.282556988648868 6.0958890871509315, axis 1 0 0, limit lower=3.1415 upper=-3.1415 effort=1 velocity=1
- added joint 313_to_210: type revolute, parent 210, child 313, origin xyz=0.9999 0.4535889622219287 0.8606944566278526 rpy=25.06201453255268 6.282556988648868 6.0958890871509315, axis 1 0 0, limit lower=3.1415 upper=-3.1415 effort=1 velocity=1
- added joint 316_to_215: type revolute, parent 215, child 316, origin xyz=0.9999 0.4535889622219287 0.8606944566278526 rpy=12.53100726627634 6.282556988648868 6.0958890871509315, axis 1 0 0, limit lower=3.1415 upper=-3.1415 effort=1 velocity=1
- added joint 317_to_215: type revolute, parent 215, child 317, origin xyz=0.9999 0.4535889622219287 0.8606944566278526 rpy=18.79651089941451 6.282556988648868 6.0958890871509315, axis 1 0 0, limit lower=3.1415 upper=-3.1415 effort=1 velocity=1
- added joint 318_to_215: type revolute, parent 215, child 318, origin xyz=0.9999 0.4535889622219287 0.8606944566278526 rpy=25.06201453255268 6.282556988648868 6.0958890871509315, axis 1 0 0, limit lower=3.1415 upper=-3.1415 effort=1 velocity=1
- added joint 320_to_219: type revolute, parent 219, child 320, origin xyz=0.9999 0.4535889622219287 0.8606944566278526 rpy=12.53100726627634 6.282556988648868 6.0958890871509315, axis 1 0 0, limit lower=3.1415 upper=-3.1415 effort=1 velocity=1
- added joint 321_to_219: type revolute, parent 219, child 321, origin xyz=0.9999 0.4535889622219287 0.8606944566278526 rpy=18.79651089941451 6.282556988648868 6.0958890871509315, axis 1 0 0, limit lower=3.1415 upper=-3.1415 effort=1 velocity=1
- added joint 322_to_219: type revolute, parent 219, child 322, origin xyz=0.9999 0.4535889622219287 0.8606944566278526 rpy=25.06201453255268 6.282556988648868 6.0958890871509315, axis 1 0 0, limit lower=3.1415 upper=-3.1415 effort=1 velocity=1
- added joint 324_to_223: type revolute, parent 223, child 324, origin xyz=0.9999 0.4535889622219287 0.8606944566278526 rpy=12.53100726627634 6.282556988648868 6.0958890871509315, axis 1 0 0, limit lower=3.1415 upper=-3.1415 effort=1 velocity=1
- added joint 325_to_223: type revolute, parent 223, child 325, origin xyz=0.9999 0.4535889622219287 0.8606944566278526 rpy=18.79651089941451 6.282556988648868 6.0958890871509315, axis 1 0 0, limit lower=3.1415 upper=-3.1415 effort=1 velocity=1
- added joint 326_to_223: type revolute, parent 223, child 326, origin xyz=0.9999 0.4535889622219287 0.8606944566278526 rpy=25.06201453255268 6.282556988648868 6.0958890871509315, axis 1 0 0, limit lower=3.1415 upper=-3.1415 effort=1 velocity=1
- added joint 329_to_228: type revolute, parent 228, child 329, origin xyz=0.9999 0.4535889622219287 0.8606944566278526 rpy=12.53100726627634 6.282556988648868 6.0958890871509315, axis 1 0 0, limit lower=3.1415 upper=-3.1415 effort=1 velocity=1
- added joint 330_to_228: type revolute, parent 228, child 330, origin xyz=0.9999 0.4535889622219287 0.8606944566278526 rpy=18.79651089941451 6.282556988648868 6.0958890871509315, axis 1 0 0, limit lower=3.1415 upper=-3.1415 effort=1 velocity=1
- added joint 331_to_228: type revolute, parent 228, child 331, origin xyz=0.9999 0.4535889622219287 0.8606944566278526 rpy=25.06201453255268 6.282556988648868 6.0958890871509315, axis 1 0 0, limit lower=3.1415 upper=-3.1415 effort=1 velocity=1
- added joint 333_to_232: type revolute, parent 232, child 333, origin xyz=0.9999 0.4535889622219287 0.8606944566278526 rpy=12.53100726627634 6.282556988648868 6.0958890871509315, axis 1 0 0, limit lower=3.1415 upper=-3.1415 effort=1 velocity=1
- added joint 334_to_232: type revolute, parent 232, child 334, origin xyz=0.9999 0.4535889622219287 0.8606944566278526 rpy=18.79651089941451 6.282556988648868 6.0958890871509315, axis 1 0 0, limit lower=3.1415 upper=-3.1415 effort=1 velocity=1
- added joint 335_to_232: type revolute, parent 232, child 335, origin xyz=0.9999 0.4535889622219287 0.8606944566278526 rpy=25.06201453255268 6.282556988648868 6.0958890871509315, axis 1 0 0, limit lower=3.1415 upper=-3.1415 effort=1 velocity=1
- added joint 337_to_236: type revolute, parent 236, child 337, origin xyz=0.9999 0.4535889622219287 0.8606944566278526 rpy=12.53100726627634 6.282556988648868 6.0958890871509315, axis 1 0 0, limit lower=3.1415 upper=-3.1415 effort=1 velocity=1
- added joint 338_to_236: type revolute, parent 236, child 338, origin xyz=0.9999 0.4535889622219287 0.8606944566278526 rpy=18.79651089941451 6.282556988648868 6.0958890871509315, axis 1 0 0, limit lower=3.1415 upper=-3.1415 effort=1 velocity=1
- added joint 339_to_236: type revolute, parent 236, child 339, origin xyz=0.9999 0.4535889622219287 0.8606944566278526 rpy=25.06201453255268 6.282556988648868 6.0958890871509315, axis 1 0 0, limit lower=3.1415 upper=-3.1415 effort=1 velocity=1
- added joint 33_to_22: type revolute, parent 22, child 33, origin xyz=0.9999 0.4535889622219287 0.8606944566278526 rpy=12.53100726627634 6.282556988648868 6.0958890871509315, axis 1 0 0, limit lower=3.1415 upper=-3.1415 effort=1 velocity=1
- added joint 34_to_22: type revolute, parent 22, child 34, origin xyz=0.9999 0.4535889622219287 0.8606944566278526 rpy=18.79651089941451 6.282556988648868 6.0958890871509315, axis 1 0 0, limit lower=3.1415 upper=-3.1415 effort=1 velocity=1
- added joint 35_to_22: type revolute, parent 22, child 35, origin xyz=0.9999 0.4535889622219287 0.8606944566278526 rpy=25.06201453255268 6.282556988648868 6.0958890871509315, axis 1 0 0, limit lower=3.1415 upper=-3.1415 effort=1 velocity=1
- added joint 37_to_26: type revolute, parent 26, child 37, origin xyz=0.9999 0.4535889622219287 0.8606944566278526 rpy=12.53100726627634 6.282556988648868 6.0958890871509315, axis 1 0 0, limit lower=3.1415 upper=-3.1415 effort=1 velocity=1
- added joint 38_to_26: type revolute, parent 26, child 38, origin xyz=0.9999 0.4535889622219287 0.8606944566278526 rpy=18.79651089941451 6.282556988648868 6.0958890871509315, axis 1 0 0, limit lower=3.1415 upper=-3.1415 effort=1 velocity=1
- added joint 39_to_26: type revolute, parent 26, child 39, origin xyz=0.9999 0.4535889622219287 0.8606944566278526 rpy=25.06201453255268 6.282556988648868 6.0958890871509315, axis 1 0 0, limit lower=3.1415 upper=-3.1415 effort=1 velocity=1
