Commit message: WOrk on project

File: midterm/part_b/source_code/my_code/test.urdf (robot description, URDF)
Before this commit: robot pepe, 5 links, 4 joints
Links:
- removed link 22
- removed link 24
- added link 12, mass 0.009384431897394841; collision cylinder length=0.584641471155833 radius=0.07147995129228524; visual cylinder length=0.584641471155833 radius=0.07147995129228524
- added link 213, mass 0.27575643462192695; collision cylinder length=0.17925070101726326 radius=0.6997734482672737; visual cylinder length=0.17925070101726326 radius=0.6997734482672737
- added link 28, mass 0.27575643462192695; collision cylinder length=0.17925070101726326 radius=0.6997734482672737; visual cylinder length=0.17925070101726326 radius=0.6997734482672737
- added link 310, mass 0.24324921543581376; collision cylinder length=0.6238276488814412 radius=0.35230473329466894; visual cylinder length=0.6238276488814412 radius=0.35230473329466894
- added link 311, mass 0.24324921543581376; collision cylinder length=0.6238276488814412 radius=0.35230473329466894; visual cylinder length=0.6238276488814412 radius=0.35230473329466894
- added link 314, mass 0.24324921543581376; collision cylinder length=0.6238276488814412 radius=0.35230473329466894; visual cylinder length=0.6238276488814412 radius=0.35230473329466894
- added link 315, mass 0.24324921543581376; collision cylinder length=0.6238276488814412 radius=0.35230473329466894; visual cylinder length=0.6238276488814412 radius=0.35230473329466894
- added link 316, mass 0.24324921543581376; collision cylinder length=0.6238276488814412 radius=0.35230473329466894; visual cylinder length=0.6238276488814412 radius=0.35230473329466894
- added link 34, mass 0.24324921543581376; collision cylinder length=0.6238276488814412 radius=0.35230473329466894; visual cylinder length=0.6238276488814412 radius=0.35230473329466894
- added link 35, mass 0.24324921543581376; collision cylinder length=0.6238276488814412 radius=0.35230473329466894; visual cylinder length=0.6238276488814412 radius=0.35230473329466894
- added link 36, mass 0.24324921543581376; collision cylinder length=0.6238276488814412 radius=0.35230473329466894; visual cylinder length=0.6238276488814412 radius=0.35230473329466894
- added link 39, mass 0.24324921543581376; collision cylinder length=0.6238276488814412 radius=0.35230473329466894; visual cylinder length=0.6238276488814412 radius=0.35230473329466894
- added link 412, mass 0.6232700589160848; collision cylinder length=0.3124077720341125 radius=0.7968971636183612; visual cylinder length=0.3124077720341125 radius=0.7968971636183612
- added link 417, mass 0.6232700589160848; collision cylinder length=0.3124077720341125 radius=0.7968971636183612; visual cylinder length=0.3124077720341125 radius=0.7968971636183612
- added link 47, mass 0.6232700589160848; collision cylinder length=0.3124077720341125 radius=0.7968971636183612; visual cylinder length=0.3124077720341125 radius=0.7968971636183612
- link 0: mass 2.5930331903046304 -> 0.05446562338846407; geometry collision cylinder length=0.07893186848787903 radius=0.46866239893441386; visual cylinder length=0.07893186848787903 radius=0.46866239893441386
- link 11: mass 0.358686335824467 -> 0.009384431897394841; geometry collision cylinder length=0.584641471155833 radius=0.07147995129228524; visual cylinder length=0.584641471155833 radius=0.07147995129228524
- link 23: mass 6.281300540076709 -> 0.27575643462192695; geometry collision cylinder length=0.17925070101726326 radius=0.6997734482672737; visual cylinder length=0.17925070101726326 radius=0.6997734482672737
Joints:
- removed joint 22_to_11
- removed joint 23_to_11
- removed joint 24_to_11
- added joint 12_to_0: type revolute, parent 0, child 12, origin xyz=0.5903723918258782 0.27126609059194107 0.411340176856842 rpy=2.4297555315444708 5.039879185013631 1.092108061001404, axis 1 0 0, limit lower=3.1415 upper=-3.1415 effort=1 velocity=1
- added joint 213_to_0: type revolute, parent 0, child 213, origin xyz=0.5376772300806993 0.603124008151945 0.8344095790129977 rpy=28.79871923746301 1.4897510611477551 5.694090256298467, axis 0 0 1, limit lower=3.1415 upper=-3.1415 effort=1 velocity=1
- added joint 23_to_0: type revolute, parent 0, child 23, origin xyz=0.5376772300806993 0.603124008151945 0.8344095790129977 rpy=19.199146158308675 1.4897510611477551 5.694090256298467, axis 0 0 1, limit lower=3.1415 upper=-3.1415 effort=1 velocity=1
- added joint 28_to_0: type revolute, parent 0, child 28, origin xyz=0.5376772300806993 0.603124008151945 0.8344095790129977 rpy=23.998932697885845 1.4897510611477551 5.694090256298467, axis 0 0 1, limit lower=3.1415 upper=-3.1415 effort=1 velocity=1
- added joint 310_to_28: type revolute, parent 28, child 310, origin xyz=0.9547207298280475 0.12961233736711997 0.11781820841747281 rpy=16.765187939652115 1.2145000660662921 0.24739232592759544, axis 1 0 0, limit lower=3.1415 upper=-3.1415 effort=1 velocity=1
- added joint 311_to_28: type revolute, parent 28, child 311, origin xyz=0.9547207298280475 0.12961233736711997 0.11781820841747281 rpy=22.353583919536153 1.2145000660662921 0.24739232592759544, axis 1 0 0, limit lower=3.1415 upper=-3.1415 effort=1 velocity=1
- added joint 314_to_213: type revolute, parent 213, child 314, origin xyz=0.9547207298280475 0.12961233736711997 0.11781820841747281 rpy=11.176791959768076 1.2145000660662921 0.24739232592759544, axis 1 0 0, limit lower=3.1415 upper=-3.1415 effort=1 velocity=1
- added joint 315_to_213: type revolute, parent 213, child 315, origin xyz=0.9547207298280475 0.12961233736711997 0.11781820841747281 rpy=16.765187939652115 1.2145000660662921 0.24739232592759544, axis 1 0 0, limit lower=3.1415 upper=-3.1415 effort=1 velocity=1
- added joint 316_to_213: type revolute, parent 213, child 316, origin xyz=0.9547207298280475 0.12961233736711997 0.11781820841747281 rpy=22.353583919536153 1.2145000660662921 0.24739232592759544, axis 1 0 0, limit lower=3.1415 upper=-3.1415 effort=1 velocity=1
- added joint 34_to_23: type revolute, parent 23, child 34, origin xyz=0.9547207298280475 0.12961233736711997 0.11781820841747281 rpy=11.176791959768076 1.2145000660662921 0.24739232592759544, axis 1 0 0, limit lower=3.1415 upper=-3.1415 effort=1 velocity=1
- added joint 35_to_23: type revolute, parent 23, child 35, origin xyz=0.9547207298280475 0.12961233736711997 0.11781820841747281 rpy=16.765187939652115 1.2145000660662921 0.24739232592759544, axis 1 0 0, limit lower=3.1415 upper=-3.1415 effort=1 velocity=1
- added joint 36_to_23: type revolute, parent 23, child 36, origin xyz=0.9547207298280475 0.12961233736711997 0.11781820841747281 rpy=22.353583919536153 1.2145000660662921 0.24739232592759544, axis 1 0 0, limit lower=3.1415 upper=-3.1415 effort=1 velocity=1
- added joint 39_to_28: type revolute, parent 28, child 39, origin xyz=0.9547207298280475 0.12961233736711997 0.11781820841747281 rpy=11.176791959768076 1.2145000660662921 0.24739232592759544, axis 1 0 0, limit lower=3.1415 upper=-3.1415 effort=1 velocity=1
- added joint 412_to_28: type revolute, parent 28, child 412, origin xyz=0.28565147263700275 0.9190752028033 0.017783262352058737 rpy=27.625929851087992 5.151798869063974 4.8569872961964, axis 1 0 0, limit lower=3.1415 upper=-3.1415 effort=1 velocity=1
- added joint 417_to_213: type revolute, parent 213, child 417, origin xyz=0.28565147263700275 0.9190752028033 0.017783262352058737 rpy=27.625929851087992 5.151798869063974 4.8569872961964, axis 1 0 0, limit lower=3.1415 upper=-3.1415 effort=1 velocity=1
- added joint 47_to_23: type revolute, parent 23, child 47, origin xyz=0.28565147263700275 0.9190752028033 0.017783262352058737 rpy=27.625929851087992 5.151798869063974 4.8569872961964, axis 1 0 0, limit lower=3.1415 upper=-3.1415 effort=1 velocity=1
- joint 11_to_0: origin xyz=0.3460188446689044 0.6833411772002934 0.7033764135855681 rpy=9.077885448262554 1.0902438349063948 0.6867123107155225 -> xyz=0.5903723918258782 0.27126609059194107 0.411340176856842 rpy=1.6198370210296473 5.039879185013631 1.092108061001404

Commit message: Shapes added

File: midterm/part_b/source_code/my_code/temp0.urdf (robot description, URDF)
Before this commit: robot pepe, 40 links, 39 joints
Links:
- removed link 114
- removed link 127
- removed link 210
- removed link 215
- removed link 219
- removed link 223
- removed link 228
- removed link 232
- removed link 236
- removed link 26
- removed link 311
- removed link 312
- removed link 313
- removed link 316
- removed link 317
- removed link 318
- removed link 320
- removed link 321
- removed link 322
- removed link 324
- removed link 325
- removed link 326
- removed link 329
- removed link 33
- removed link 330
- removed link 331
- removed link 333
- removed link 334
- removed link 335
- removed link 337
- removed link 338
- removed link 339
- removed link 34
- removed link 35
- removed link 37
- removed link 38
- removed link 39
- added link 23, mass 0.002794580386715296; collision cylinder length=0.33092395444948486 radius=0.051846478571480725; visual cylinder length=0.33092395444948486 radius=0.051846478571480725
- link 0: mass 0.16089181704610028 -> 1.1506211025735562; geometry collision cylinder length=0.5625772901796258 radius=0.8068636167950674; visual cylinder length=0.5625772901796258 radius=0.8068636167950674
- link 11: mass 6.0568130706387295 -> 0.40020041811534046; geometry collision cylinder length=0.35441705586968714 radius=0.599523934459773; visual cylinder length=0.35441705586968714 radius=0.599523934459773
- link 22: mass 6.0568130706387295 -> 0.002794580386715296; geometry collision cylinder length=0.33092395444948486 radius=0.051846478571480725; visual cylinder length=0.33092395444948486 radius=0.051846478571480725
Joints:
- removed joint 114_to_0
- removed joint 127_to_0
- removed joint 210_to_11
- removed joint 215_to_114
- removed joint 219_to_114
- removed joint 223_to_114
- removed joint 228_to_127
- removed joint 232_to_127
- removed joint 236_to_127
- removed joint 26_to_11
- removed joint 311_to_210
- removed joint 312_to_210
- removed joint 313_to_210
- removed joint 316_to_215
- removed joint 317_to_215
- removed joint 318_to_215
- removed joint 320_to_219
- removed joint 321_to_219
- removed joint 322_to_219
- removed joint 324_to_223
- removed joint 325_to_223
- removed joint 326_to_223
- removed joint 329_to_228
- removed joint 330_to_228
- removed joint 331_to_228
- removed joint 333_to_232
- removed joint 334_to_232
- removed joint 335_to_232
- removed joint 337_to_236
- removed joint 338_to_236
- removed joint 339_to_236
- removed joint 33_to_22
- removed joint 34_to_22
- removed joint 35_to_22
- removed joint 37_to_26
- removed joint 38_to_26
- removed joint 39_to_26
- added joint 23_to_11: type revolute, parent 11, child 23, origin xyz=0.9999 0.3204026496109833 0.6642333311931486 rpy=16.66211687380712 3.4606752119847273 0.5377040303247361, axis 0 0 1, limit lower=3.1415 upper=-3.1415 effort=1 velocity=1
- joint 11_to_0: axis 1 0 0 -> 0 0 1; origin xyz=0.9999 0.3535889622219287 0.9606944566278526 rpy=11.274370204840425 6.282556988648868 6.0958890871509315 -> xyz=0.6287796269892859 0.4798738006784883 0.6636635622644665 rpy=9.519351475367962 1.7503012391596664 2.2361916503454458
- joint 22_to_11: axis 1 0 0 -> 0 0 1; origin xyz=0.864255060277676 0.7535889622219286 0.8606944566278526 rpy=10.017733143404508 5.356506984867917 6.0958890871509315 -> xyz=0.9999 0.3204026496109833 0.6642333311931486 rpy=11.108077915871412 3.4606752119847273 0.5377040303247361

File: midterm/part_b/source_code/my_code/test.urdf (robot description, URDF)
Before this commit: robot pepe, 18 links, 17 joints
Links:
- removed link 12
- removed link 213
- removed link 23
- removed link 28
- removed link 310
- removed link 311
- removed link 314
- removed link 315
- removed link 316
- removed link 34
- removed link 35
- removed link 36
- removed link 39
- removed link 412
- removed link 417
- removed link 47
- added link 13, mass 1.1506211025735562; collision cylinder length=0.5625772901796258 radius=0.8068636167950674; visual cylinder length=0.5625772901796258 radius=0.8068636167950674
- added link 15, mass 1.1506211025735562; collision cylinder length=0.5625772901796258 radius=0.8068636167950674; visual cylinder length=0.5625772901796258 radius=0.8068636167950674
- added link 22, mass 0.1743645496166827; collision cylinder length=0.15441705586968713 radius=0.599523934459773; visual cylinder length=0.15441705586968713 radius=0.599523934459773
- added link 24, mass 0.1743645496166827; collision cylinder length=0.15441705586968713 radius=0.599523934459773; visual cylinder length=0.15441705586968713 radius=0.599523934459773
- added link 26, mass 0.1743645496166827; collision cylinder length=0.15441705586968713 radius=0.599523934459773; visual cylinder length=0.15441705586968713 radius=0.599523934459773
- link 0: mass 0.05446562338846407 -> 0.0006491701219059603; geometry collision cylinder length=1.1226638615419493 radius=0.013566863446804911; visual cylinder length=1.1226638615419493 radius=0.013566863446804911
- link 11: mass 0.009384431897394841 -> 1.1506211025735562; geometry collision cylinder length=0.5625772901796258 radius=0.8068636167950674; visual cylinder length=0.5625772901796258 radius=0.8068636167950674
Joints:
- removed joint 12_to_0
- removed joint 213_to_0
- removed joint 23_to_0
- removed joint 28_to_0
- removed joint 310_to_28
- removed joint 311_to_28
- removed joint 314_to_213
- removed joint 315_to_213
- removed joint 316_to_213
- removed joint 34_to_23
- removed joint 35_to_23
- removed joint 36_to_23
- removed joint 39_to_28
- removed joint 412_to_28
- removed joint 417_to_213
- removed joint 47_to_23
- added joint 13_to_0: type revolute, parent 0, child 13, origin xyz=0.18977128553073197 0.5336053814382133 0.17036618091553735 rpy=7.08169284061338 1.9845007485072967 1.53768567894434, axis 0 0 1, limit lower=3.1415 upper=-3.1415 effort=1 velocity=1
- added joint 15_to_0: type revolute, parent 0, child 15, origin xyz=0.18977128553073197 0.5336053814382133 0.17036618091553735 rpy=9.44225712081784 1.9845007485072967 1.53768567894434, axis 0 0 1, limit lower=3.1415 upper=-3.1415 effort=1 velocity=1
- added joint 22_to_11: type revolute, parent 11, child 22, origin xyz=0.6287796269892859 0.4798738006784883 0.6636635622644665 rpy=9.519351475367962 1.7503012391596664 1.6078731196274874, axis 0 0 1, limit lower=3.1415 upper=-3.1415 effort=1 velocity=1
- added joint 24_to_13: type revolute, parent 13, child 24, origin xyz=0.6287796269892859 0.4798738006784883 0.6636635622644665 rpy=9.519351475367962 1.7503012391596664 1.6078731196274874, axis 0 0 1, limit lower=3.1415 upper=-3.1415 effort=1 velocity=1
- added joint 26_to_15: type revolute, parent 15, child 26, origin xyz=0.6287796269892859 0.4798738006784883 0.6636635622644665 rpy=9.519351475367962 1.7503012391596664 1.6078731196274874, axis 0 0 1, limit lower=3.1415 upper=-3.1415 effort=1 velocity=1
- joint 11_to_0: axis 1 0 0 -> 0 0 1; origin xyz=0.5903723918258782 0.27126609059194107 0.411340176856842 rpy=1.6198370210296473 5.039879185013631 1.092108061001404 -> xyz=0.18977128553073197 0.5336053814382133 0.17036618091553735 rpy=4.72112856040892 1.9845007485072967 1.53768567894434
